Commit message: removed the front laser scanner from the model since we do not have it

File: workspaces/youbot/src/youbot_description/urdf/youbot_base/base.urdf.xacro (robot description, xacro)
@@ -84,5 +84,5 @@
 		<!-- base laser front -->
     		<xacro:hokuyo_urg04_laser name="${name}_laser_front" parent="${name}" ros_topic="scan_front" update_rate="10" min_angle="-1.57" max_angle="1.57" >
-     			 <origin xyz="0.3 0 -0.03" rpy="3.14 0 0" />
+     			 <origin xyz="0.3 0 -0.03" rpy="0 0 0" />
     		</xacro:hokuyo_urg04_laser>
 	<!-- front left wheel -->
