Commit message: Full Base IK planner, with 8 DOF

File: workspaces/youbot/src/youbot_description/urdf/youbot_base/base_within_IK.urdf.xacro (robot description, xacro)
@@ -55,18 +55,35 @@
       			</collision>
     		</link>
-		<link name="base_dummy_link">
+		<link name="base_dummy_prismatic_x_link">
 		</link>
-		<joint name="${name}_footprint_joint" type="revolute">
+		<link name="base_dummy_prismatic_y_link">
+		</link>
+		<link name="base_dummy_revolute_link">
+		</link>
+		<joint name="${name}_footprint_joint" type="fixed">
+      			<origin xyz="0 0 0" rpy="0 0 0" />
+      			<child link="base_dummy_revolute_link" />
+      			<parent link="${name}_footprint"/>
+    		</joint>
+		<joint name="base_dummy_revolute_joint" type="revolute">
       			<origin xyz="0 0 0" rpy="0 0 0" />
 			<axis xyz="0 0 1" />
-			<child link="base_dummy_link" />
-      			<parent link="${name}_footprint"/>
+			<child link="base_dummy_prismatic_x_link" />
+      			<parent link="base_dummy_revolute_link"/>
 			<limit effort="${9.5}" velocity="${M_PI}" lower="${-M_PI}" upper="${M_PI}"/>
     		</joint>
-		<joint name="base_dummy_joint" type="prismatic">
+		<joint name="base_dummy_prismatic_x_joint" type="prismatic">
       			<origin xyz="0 0 0" rpy="0 0 0" />
+			<axis xyz="1 0 0" />
+			<child link="base_dummy_prismatic_y_link" />
+      			<parent link="base_dummy_prismatic_x_link"/>
+			<limit effort="${9.5}" velocity="${M_PI}" lower="${-50}" upper="${50}"/>
+    		</joint>
+		<joint name="base_dummy_prismatic_y_joint" type="prismatic">
+      			<origin xyz="0 0 0" rpy="0 0 0" />
+			<axis xyz="0 1 0" />
 			<child link="${name}_link" />
-      			<parent link="base_dummy_link"/>
-			<limit effort="${9.5}" velocity="${M_PI}" lower="${-100}" upper="${100}"/>
+      			<parent link="base_dummy_prismatic_y_link"/>
+			<limit effort="${9.5}" velocity="${M_PI}" lower="${-50}" upper="${50}"/>
     		</joint>
 		<link name="${name}_link">

Commit message: Signed-off-by: yiming <yymalex@gmail.com>

File: workspaces/youbot/src/youbot_description/urdf/youbot_base/base_within_IK.urdf.xacro (robot description, xacro)
@@ -55,4 +55,6 @@
       			</collision-->
     		</link>
+		<link name ="moveit_fixed_link">
+		</link>
 		<link name="${name}_link">
       			<inertial>
@@ -119,4 +121,9 @@
       			</collision>
 		</link>
+		<joint name="moveit_fixed_joint" type="fixed">
+			<origin xyz="0 0 0" rpy="0 0 0" />
+			<child link="moveit_fixed_link"/>
+			<parent link="${name}_footprint" />
+		</joint>
 		<joint name="dummy_prismatic_x_joint" type="prismatic">
 			<origin xyz="0 0 0" rpy="0 0 0" />
@@ -124,5 +131,5 @@
 			<limit effort="${9.5}" velocity="${M_PI}" lower="${-50}" upper="${50}"/>
       			<child link="dummy_prismatic_link" />
-      			<parent link="${name}_footprint"/>
+      			<parent link="moveit_fixed_link"/>
     		</joint>
 		<joint name="dummy_prismatic_y_joint" type="prismatic">

Commit message: Signed-off-by: yiming <yymalex@gmail.com>

File: workspaces/youbot/src/youbot_description/urdf/youbot_base/base_within_IK.urdf.xacro (robot description, xacro)
@@ -72,52 +72,14 @@
       			</visual>
       			<collision>
-        			<origin xyz="0 0 0" rpy="0 0 0" />
-        			<geometry>
-          				<!--<box size="${base_size_x} ${base_size_y} ${base_size_z}" />-->
-					<mesh filename="package://youbot_description/meshes/youbot_base/base_convex.dae"/>
+        			<origin xyz="0 0 0.05" rpy="0 0 0" />
+        			<geometry>
+          				<box size="${base_size_x} ${base_size_y} ${base_size_z}" />
+					<!--mesh filename="package://youbot_description/meshes/youbot_base/base_convex.dae"/-->
 	       			</geometry>
       			</collision>
     		</link>
 		<link name="dummy_prismatic_link">
-			<inertial>
-        			<mass value="0.0001" />
-        			<origin xyz="0 0 ${-base_size_z / 2.0}" rpy="0 0 0" />
-        			<inertia ixx="1.0" ixy="0.0" ixz="0.0"
-                 			iyy="1.0" iyz="0.0" izz="1.0" />
-      				</inertial>
-      			<visual>
-        			<origin xyz="0 0 0" rpy="0 0 0" />
-        			<geometry>
-          				<box size="0.001 0.001 0.001" />
-        			</geometry>
-               			<material name="Red" />
-      			</visual>
-      			<collision>
-        			<origin xyz="0 0 ${-base_size_z / 2.0}" rpy="0 0 0" />
-        			<geometry>
-          				<box size="0.001 0.001 0.001" />
-        			</geometry>
-      			</collision>
 		</link>
 		<link name="dummy_revolute_link">
-			<inertial>
-        			<mass value="0.0001" />
-        			<origin xyz="0 0 ${-base_size_z / 2.0}" rpy="0 0 0" />
-        			<inertia ixx="1.0" ixy="0.0" ixz="0.0"
-                 			iyy="1.0" iyz="0.0" izz="1.0" />
-      				</inertial>
-      			<visual>
-        			<origin xyz="0 0 0" rpy="0 0 0" />
-        			<geometry>
-          				<box size="0.001 0.001 0.001" />
-        			</geometry>
-               			<material name="Red" />
-      			</visual>
-      			<collision>
-        			<origin xyz="0 0 ${-base_size_z / 2.0}" rpy="0 0 0" />
-        			<geometry>
-          				<box size="0.001 0.001 0.001" />
-        			</geometry>
-      			</collision>
 		</link>
 		<joint name="moveit_fixed_joint" type="fixed">
@@ -129,5 +91,5 @@
 			<origin xyz="0 0 0" rpy="0 0 0" />
 			<axis xyz="1 0 0" />
-			<limit effort="${9.5}" velocity="${M_PI}" lower="${-50}" upper="${50}"/>
+			<limit effort="${9.5}" velocity="${M_PI}" lower="${-10}" upper="${10}"/>
       			<child link="dummy_prismatic_link" />
       			<parent link="moveit_fixed_link"/>
@@ -138,5 +100,5 @@
 			<child link="dummy_revolute_link" />
       			<parent link="dummy_prismatic_link"/>
-			<limit effort="${9.5}" velocity="${M_PI}" lower="${-50}" upper="${50}"/>
+			<limit effort="${9.5}" velocity="${M_PI}" lower="${-10}" upper="${10}"/>
     		</joint>
 		<joint name="dummy_revolute_joint" type="revolute">
@@ -193,5 +155,5 @@
       			</visual>
       			<collision>
-        			<origin xyz="0 0 0" rpy="${M_PI/2} 0 0" />
+        			<origin xyz="0 0 0.05" rpy="${M_PI/2} 0 0" />
         			<geometry>
         		       		<cylinder radius="${wheel_radius}" length="${wheel_radius}" />
@@ -241,5 +203,5 @@
       			</visual>
       			<collision>
-        			<origin xyz="0 0 0" rpy="${M_PI/2} 0 0" />
+        			<origin xyz="0 0 0.05" rpy="${M_PI/2} 0 0" />
         			<geometry>
         		       		<cylinder radius="${wheel_radius}" length="${wheel_radius}" />
@@ -290,5 +252,5 @@
       			</visual>
       			<collision>
-        			<origin xyz="0 0 0" rpy="${M_PI/2} 0 0" />
+        			<origin xyz="0 0 0.05" rpy="${M_PI/2} 0 0" />
         			<geometry>
         		       		<cylinder radius="${wheel_radius}" length="${wheel_radius}" />
@@ -341,5 +303,5 @@
       			</visual>
       			<collision>
-        			<origin xyz="0 0 0" rpy="${M_PI/2} 0 0" />
+        			<origin xyz="0 0 0.05" rpy="${M_PI/2} 0 0" />
         			<geometry>
         		       		<cylinder radius="${wheel_radius}" length="${wheel_radius}" />

Commit message: Signed-off-by: yiming <yymalex@gmail.com>

File: workspaces/youbot/src/youbot_description/urdf/youbot_base/base_within_IK.urdf.xacro (robot description, xacro)
@@ -72,5 +72,5 @@
       			</visual>
       			<collision>
-        			<origin xyz="0 0 0.05" rpy="0 0 0" />
+        			<origin xyz="0 0 0.0" rpy="0 0 0" />
         			<geometry>
           				<box size="${base_size_x} ${base_size_y} ${base_size_z}" />
@@ -155,5 +155,5 @@
       			</visual>
       			<collision>
-        			<origin xyz="0 0 0.05" rpy="${M_PI/2} 0 0" />
+        			<origin xyz="0 0 0.0" rpy="${M_PI/2} 0 0" />
         			<geometry>
         		       		<cylinder radius="${wheel_radius}" length="${wheel_radius}" />
@@ -203,5 +203,5 @@
       			</visual>
       			<collision>
-        			<origin xyz="0 0 0.05" rpy="${M_PI/2} 0 0" />
+        			<origin xyz="0 0 0.0" rpy="${M_PI/2} 0 0" />
         			<geometry>
         		       		<cylinder radius="${wheel_radius}" length="${wheel_radius}" />
@@ -252,5 +252,5 @@
       			</visual>
       			<collision>
-        			<origin xyz="0 0 0.05" rpy="${M_PI/2} 0 0" />
+        			<origin xyz="0 0 0.0" rpy="${M_PI/2} 0 0" />
         			<geometry>
         		       		<cylinder radius="${wheel_radius}" length="${wheel_radius}" />
@@ -303,5 +303,5 @@
       			</visual>
       			<collision>
-        			<origin xyz="0 0 0.05" rpy="${M_PI/2} 0 0" />
+        			<origin xyz="0 0 0.0" rpy="${M_PI/2} 0 0" />
         			<geometry>
         		       		<cylinder radius="${wheel_radius}" length="${wheel_radius}" />
