Commit message: link name change

File: workspaces/youbot/src/youbot_description/urdf/sensors/asus_xtion_camera.urdf.xacro (robot description, xacro)
@@ -5,5 +5,5 @@
         xmlns:xacro="http://ros.org/wiki/xacro">
   <property name="M_PI" value="3.14159"/>.
-  <include filename="$(find youbot_description)/urdf/sensors/asus_xtion_camera.gazebo.xacro" />
+  <include filename="$(find youbot_description)/urdf/sensors/asus_xtion_link.gazebo.xacro" />
   <property name="eye_x_offset" value="0.03" />
   <property name="eye_y_offset" value="0.035" />
@@ -17,11 +17,11 @@
 	</link>
 	<joint name="${parent}_${suffix}_joint" type="fixed">
-	  <parent link="${parent}_camera"/>
+	  <parent link="${parent}_link"/>
 	  <child link="${parent}_${suffix}_frame"/>
 	  <insert_block name="origin"/>
 	</joint>
   </xacro:macro>
-  <xacro:macro name="asus_xtion_camera" params="name parent *origin tilt">
-    <link name="${name}_camera">
+  <xacro:macro name="asus_xtion_link" params="name parent *origin tilt">
+    <link name="${name}_link">
       <inertial>
         <mass value="0.1" />
@@ -32,5 +32,5 @@
         <origin xyz="0.02 -0.03 0" rpy="${M_PI/2} 0 ${M_PI/2}" />
         <geometry>
-          <mesh filename="package://youbot_description/meshes/sensors/asus_xtion_pro_live_camera.dae" scale="0.001 0.001 0.001"/>
+          <mesh filename="package://youbot_description/meshes/sensors/asus_xtion_pro_live_link.dae" scale="0.001 0.001 0.001"/>
         </geometry>
         <material name="Black" />
@@ -41,5 +41,5 @@
    	  <box size="0.2 0.06 0.07"/>
 <!--
-	  <mesh filename="package://youbot_description/meshes/sensors/asus_xtion_pro_live_camera.dae" scale="0.001 0.001 0.001"/>
+	  <mesh filename="package://youbot_description/meshes/sensors/asus_xtion_pro_live_link.dae" scale="0.001 0.001 0.001"/>
 -->
         </geometry>
@@ -49,5 +49,5 @@
       <insert_block name="origin" />
       <parent link="${parent}" />
-      <child link="${name}_camera" />
+      <child link="${name}_link" />
     </joint>
 	<xacro:asus_xtion_eye suffix="depth" parent="${name}">
@@ -70,9 +70,9 @@
 	</xacro:asus_xtion_eye>
    <!-- for simulation -->
-   <xacro:asus_xtion_camera_gazebo name="${name}" />
+   <xacro:asus_xtion_link_gazebo name="${name}" />
   </xacro:macro>
-<!--  <xacro:asus_xtion_camera name="xtion" tilt="0.0">
+<!--  <xacro:asus_xtion_link name="xtion" tilt="0.0">
      <origin xyz="0 0 0" rpy="0 0 0" />
-  </xacro:asus_xtion_camera>
+  </xacro:asus_xtion_link>
 -->
 </robot>

Commit message: trying to fix xtion frames

File: workspaces/youbot/src/youbot_description/urdf/sensors/asus_xtion_camera.urdf.xacro (robot description, xacro)
@@ -76,3 +76,4 @@
   </xacro:asus_xtion_link>
 -->
+  </xacro:macro>
 </robot>

Commit message: improvd description in asus xacro file

File: workspaces/youbot/src/youbot_description/urdf/sensors/asus_xtion_camera.urdf.xacro (robot description, xacro)
@@ -71,9 +71,8 @@
    <!-- for simulation -->
    <xacro:asus_xtion_link_gazebo name="${name}" />
-  </xacro:macro>
+  </xacro:macro> <!--xacro:macro name="asus_xtion_link -->
 <!--  <xacro:asus_xtion_link name="xtion" tilt="0.0">
      <origin xyz="0 0 0" rpy="0 0 0" />
   </xacro:asus_xtion_link>
 -->
-  </xacro:macro>
 </robot>

Commit message: fixed dae link

File: workspaces/youbot/src/youbot_description/urdf/sensors/asus_xtion_camera.urdf.xacro (robot description, xacro)
@@ -32,5 +32,5 @@
         <origin xyz="0.02 -0.03 0" rpy="${M_PI/2} 0 ${M_PI/2}" />
         <geometry>
-          <mesh filename="package://youbot_description/meshes/sensors/asus_xtion_pro_live_link.dae" scale="0.001 0.001 0.001"/>
+          <mesh filename="package://youbot_description/meshes/sensors/asus_xtion_pro_live_camera.dae" scale="0.001 0.001 0.001"/>
         </geometry>
         <material name="Black" />
