Commit message: fixed hydro xacro:include

File: workspaces/youbot/src/youbot_description/robots/youbot-sensors.urdf.xacro (robot description, xacro)
@@ -7,17 +7,17 @@
   <!-- The following included files set up definitions of parts of the robot body -->
   <!-- misc common stuff? -->
-  <include filename="$(find youbot_description)/urdf/common.xacro" />
+  <xacro:include filename="$(find youbot_description)/urdf/common.xacro" />
   <!-- youbot base -->
-  <include filename="$(find youbot_description)/urdf/youbot_base/base.urdf.xacro" />
+  <xacro:include filename="$(find youbot_description)/urdf/youbot_base/base.urdf.xacro" />
   <!-- youbot plate -->
-  <include filename="$(find youbot_description)/urdf/youbot_plate/plate.urdf.xacro" />
+  <xacro:include filename="$(find youbot_description)/urdf/youbot_plate/plate.urdf.xacro" />
   <!-- youbot arm -->
-  <include filename="$(find youbot_description)/urdf/youbot_arm/arm.urdf.xacro"/>
+  <xacro:include filename="$(find youbot_description)/urdf/youbot_arm/arm.urdf.xacro"/>
   <!-- youbot gripper -->
-  <include filename="$(find youbot_description)/urdf/youbot_gripper/gripper.urdf.xacro" />
+  <xacro:include filename="$(find youbot_description)/urdf/youbot_gripper/gripper.urdf.xacro" />
   <!-- generic simulator_gazebo plugins for starting mechanism control, ros time, ros battery -->
-  <include filename="$(find youbot_description)/gazebo/gazebo.urdf.xacro" />
+  <xacro:include filename="$(find youbot_description)/gazebo/gazebo.urdf.xacro" />
   <!-- materials for visualization -->
-  <include filename="$(find youbot_description)/urdf/materials.urdf.xacro" />
+  <xacro:include filename="$(find youbot_description)/urdf/materials.urdf.xacro" />
   <!-- Now we can start using the macros included above to define the actual youbot -->
   <!-- The first use of a macro.  This one was defined in base.urdf.xacro above.
@@ -40,10 +40,10 @@
   </xacro:youbot_gripper>
   <!-- BRSU SPECIFIC STUFF -->
-  <include filename="$(find youbot_description)/urdf/updated_materials.urdf.xacro" />
-  <include filename="$(find youbot_description)/urdf/misc/sensor_angle.urdf.xacro" />
-  <include filename="$(find youbot_description)/urdf/misc/cam3d_tower.urdf.xacro" />
-  <include filename="$(find youbot_description)/urdf/sensors/kinect_camera.urdf.xacro" />
-  <include filename="$(find youbot_description)/urdf/sensors/microsoft_lifecam.urdf.xacro" />
-  <include filename="$(find youbot_description)/urdf/sensors/asus_xtion_camera.urdf.xacro" />
+  <xacro:include filename="$(find youbot_description)/urdf/updated_materials.urdf.xacro" />
+  <xacro:include filename="$(find youbot_description)/urdf/misc/sensor_angle.urdf.xacro" />
+  <xacro:include filename="$(find youbot_description)/urdf/misc/cam3d_tower.urdf.xacro" />
+  <xacro:include filename="$(find youbot_description)/urdf/sensors/kinect_camera.urdf.xacro" />
+  <xacro:include filename="$(find youbot_description)/urdf/sensors/microsoft_lifecam.urdf.xacro" />
+  <xacro:include filename="$(find youbot_description)/urdf/sensors/asus_xtion_camera.urdf.xacro" />
   <!-- base laser rear -->
   <xacro:hokuyo_urg04_laser name="base_laser_rear" parent="base" ros_topic="scan_rear" update_rate="10" min_angle="-1.57" max_angle="1.57">

File: workspaces/youbot/src/youbot_description/robots/youbot.urdf.xacro (robot description, xacro)
@@ -7,17 +7,17 @@
   <!-- The following included files set up definitions of parts of the robot body -->
   <!-- misc common stuff? -->
-  <include filename="$(find youbot_description)/urdf/common.xacro" />
+  <xacro:include filename="$(find youbot_description)/urdf/common.xacro" />
   <!-- youbot base -->
-  <include filename="$(find youbot_description)/urdf/youbot_base/base.urdf.xacro" />
+  <xacro:include filename="$(find youbot_description)/urdf/youbot_base/base.urdf.xacro" />
   <!-- youbot plate -->
-  <include filename="$(find youbot_description)/urdf/youbot_plate/plate.urdf.xacro" />
+  <xacro:include filename="$(find youbot_description)/urdf/youbot_plate/plate.urdf.xacro" />
   <!-- youbot arm -->
-  <include filename="$(find youbot_description)/urdf/youbot_arm/arm.urdf.xacro"/>
+  <xacro:include filename="$(find youbot_description)/urdf/youbot_arm/arm.urdf.xacro"/>
   <!-- youbot gripper -->
-  <include filename="$(find youbot_description)/urdf/youbot_gripper/gripper.urdf.xacro" />
+  <xacro:include filename="$(find youbot_description)/urdf/youbot_gripper/gripper.urdf.xacro" />
   <!-- generic simulator_gazebo plugins for starting mechanism control, ros time, ros battery -->
-  <include filename="$(find youbot_description)/gazebo/gazebo.urdf.xacro" />
+  <xacro:include filename="$(find youbot_description)/gazebo/gazebo.urdf.xacro" />
   <!-- materials for visualization -->
-  <include filename="$(find youbot_description)/urdf/materials.urdf.xacro" />
+  <xacro:include filename="$(find youbot_description)/urdf/materials.urdf.xacro" />
   <!-- Now we can start using the macros included above to define the actual youbot -->
   <!-- The first use of a macro.  This one was defined in base.urdf.xacro above.
@@ -51,10 +51,10 @@
   </xacro:youbot_plate>
 <!-- SENSOR SPECIFIC STUFF -->
-  <include filename="$(find youbot_description)/urdf/updated_materials.urdf.xacro" />
-  <include filename="$(find youbot_description)/urdf/misc/sensor_angle.urdf.xacro" />
-<!--  <include filename="$(find youbot_description)/urdf/misc/cam3d_tower.urdf.xacro" /> -->
-<!--  <include filename="$(find youbot_description)/urdf/sensors/kinect_camera.urdf.xacro" /> -->
-<!--  <include filename="$(find youbot_description)/urdf/sensors/microsoft_lifecam.urdf.xacro" /> -->
-  <include filename="$(find youbot_description)/urdf/sensors/asus_xtion_camera.urdf.xacro" />
+  <xacro:include filename="$(find youbot_description)/urdf/updated_materials.urdf.xacro" />
+  <xacro:include filename="$(find youbot_description)/urdf/misc/sensor_angle.urdf.xacro" />
+<!--  <xacro:include filename="$(find youbot_description)/urdf/misc/cam3d_tower.urdf.xacro" /> -->
+<!--  <xacro:include filename="$(find youbot_description)/urdf/sensors/kinect_camera.urdf.xacro" /> -->
+<!--  <xacro:include filename="$(find youbot_description)/urdf/sensors/microsoft_lifecam.urdf.xacro" /> -->
+  <xacro:include filename="$(find youbot_description)/urdf/sensors/asus_xtion_camera.urdf.xacro" />
   <!-- base laser rear -->
 <!--
@@ -70,5 +70,5 @@
   <xacro:asus_xtion_link name="xtion" parent="arm_sensor_angle_part2_link"  tilt="0.0">
   <!-- AR_CALIBRATOR:EDIT_HERE -->
-                  <origin xyz="-0.0256356 0.0275046 -0.0475053" rpy="3.14097 -0.273895 -3.1287" />
+                  <origin xyz="-0.0253595 0.0305853 -0.0469736" rpy="3.13948 -0.306551 -3.13083" />
   </xacro:asus_xtion_link>
 </robot>

File: workspaces/youbot/src/youbot_description/robots/youbot_arm.urdf.xacro (robot description, xacro)
@@ -7,13 +7,13 @@
   <!-- The following included files set up definitions of parts of the robot body -->
   <!-- misc common stuff? -->
-  <include filename="$(find youbot_description)/urdf/common.xacro" />
+  <xacro:include filename="$(find youbot_description)/urdf/common.xacro" />
   <!-- materials for visualization -->
-  <include filename="$(find youbot_description)/urdf/materials.urdf.xacro" />
+  <xacro:include filename="$(find youbot_description)/urdf/materials.urdf.xacro" />
   <!-- youbot arm -->
-  <include filename="$(find youbot_description)/urdf/youbot_arm/arm.urdf.xacro" />
+  <xacro:include filename="$(find youbot_description)/urdf/youbot_arm/arm.urdf.xacro" />
   <!-- youbot arm -->
-  <include filename="$(find youbot_description)/urdf/youbot_gripper/gripper.urdf.xacro" />
+  <xacro:include filename="$(find youbot_description)/urdf/youbot_gripper/gripper.urdf.xacro" />
   <!-- generic simulator_gazebo plugins for starting mechanism control, ros time, ros battery -->
-  <include filename="$(find youbot_description)/gazebo/gazebo.urdf.xacro" />
+  <xacro:include filename="$(find youbot_description)/gazebo/gazebo.urdf.xacro" />
   <!-- Now we can start using the macros included above to define the actual youbot -->
   <!-- The first use of a macro.  This one was defined in base.urdf.xacro above.

File: workspaces/youbot/src/youbot_description/robots/youbot_arm.urdf__OLD__.xacro (robot description, xacro)
@@ -7,13 +7,13 @@
   <!-- The following included files set up definitions of parts of the robot body -->
   <!-- misc common stuff? -->
-  <include filename="$(find youbot_description)/urdf/common.xacro" />
+  <xacro:include filename="$(find youbot_description)/urdf/common.xacro" />
   <!-- materials for visualization -->
-  <include filename="$(find youbot_description)/urdf/materials.urdf.xacro" />
+  <xacro:include filename="$(find youbot_description)/urdf/materials.urdf.xacro" />
   <!-- youbot arm -->
-  <include filename="$(find youbot_description)/urdf/youbot_arm/arm.urdf.xacro" />
+  <xacro:include filename="$(find youbot_description)/urdf/youbot_arm/arm.urdf.xacro" />
   <!-- youbot arm -->
-  <include filename="$(find youbot_description)/urdf/youbot_gripper/gripper.urdf.xacro" />
+  <xacro:include filename="$(find youbot_description)/urdf/youbot_gripper/gripper.urdf.xacro" />
   <!-- generic simulator_gazebo plugins for starting mechanism control, ros time, ros battery -->
-  <include filename="$(find youbot_description)/gazebo/gazebo.urdf.xacro" />
+  <xacro:include filename="$(find youbot_description)/gazebo/gazebo.urdf.xacro" />
   <!-- Now we can start using the macros included above to define the actual youbot -->
   <!-- The first use of a macro.  This one was defined in base.urdf.xacro above.

File: workspaces/youbot/src/youbot_description/robots/youbot_base.urdf.xacro (robot description, xacro)
@@ -7,11 +7,11 @@
   <!-- The following included files set up definitions of parts of the robot body -->
   <!-- misc common stuff? -->
-  <include filename="$(find youbot_description)/urdf/common.xacro" />
+  <xacro:include filename="$(find youbot_description)/urdf/common.xacro" />
   <!-- youbot base -->
-  <include filename="$(find youbot_description)/urdf/youbot_base/base.urdf.xacro" />
+  <xacro:include filename="$(find youbot_description)/urdf/youbot_base/base.urdf.xacro" />
   <!-- generic simulator_gazebo plugins for starting mechanism control, ros time, ros battery -->
-  <include filename="$(find youbot_description)/gazebo/gazebo.urdf.xacro" />
+  <xacro:include filename="$(find youbot_description)/gazebo/gazebo.urdf.xacro" />
   <!-- materials for visualization -->
-  <include filename="$(find youbot_description)/urdf/materials.urdf.xacro" />
+  <xacro:include filename="$(find youbot_description)/urdf/materials.urdf.xacro" />
   <!-- Now we can start using the macros included above to define the actual youbot -->
   <!-- The first use of a macro.  This one was defined in base.urdf.xacro above.

File: workspaces/youbot/src/youbot_description/robots/youbot_dual_arm.urdf.xacro (robot description, xacro)
@@ -7,17 +7,17 @@
   <!-- The following included files set up definitions of parts of the robot body -->
   <!-- misc common stuff? -->
-  <include filename="$(find youbot_description)/urdf/common.xacro" />
+  <xacro:include filename="$(find youbot_description)/urdf/common.xacro" />
   <!-- youbot base -->
-  <include filename="$(find youbot_description)/urdf/youbot_base/base.urdf.xacro" />
+  <xacro:include filename="$(find youbot_description)/urdf/youbot_base/base.urdf.xacro" />
   <!-- youbot plate -->
-  <include filename="$(find youbot_description)/urdf/youbot_plate/plate.urdf.xacro" />
+  <xacro:include filename="$(find youbot_description)/urdf/youbot_plate/plate.urdf.xacro" />
   <!-- youbot arm -->
-  <include filename="$(find youbot_description)/urdf/youbot_arm/arm.urdf.xacro"/>
+  <xacro:include filename="$(find youbot_description)/urdf/youbot_arm/arm.urdf.xacro"/>
   <!-- youbot gripper -->
-  <include filename="$(find youbot_description)/urdf/youbot_gripper/gripper.urdf.xacro" />
+  <xacro:include filename="$(find youbot_description)/urdf/youbot_gripper/gripper.urdf.xacro" />
   <!-- generic simulator_gazebo plugins for starting mechanism control, ros time, ros battery -->
-  <include filename="$(find youbot_description)/gazebo/gazebo.urdf.xacro" />
+  <xacro:include filename="$(find youbot_description)/gazebo/gazebo.urdf.xacro" />
   <!-- materials for visualization -->
-  <include filename="$(find youbot_description)/urdf/materials.urdf.xacro" />
+  <xacro:include filename="$(find youbot_description)/urdf/materials.urdf.xacro" />
   <!-- Now we can start using the macros included above to define the actual youbot -->
   <!-- The first use of a macro.  This one was defined in base.urdf.xacro above.

File: workspaces/youbot/src/youbot_description/robots/youbot_gripper.urdf.xacro (robot description, xacro)
@@ -7,11 +7,11 @@
   <!-- The following included files set up definitions of parts of the robot body -->
   <!-- misc common stuff? -->
-  <include filename="$(find youbot_description)/urdf/common.xacro" />
+  <xacro:include filename="$(find youbot_description)/urdf/common.xacro" />
   <!-- youbot gripper -->
-  <include filename="$(find youbot_description)/urdf/youbot_gripper/gripper.urdf.xacro" />
+  <xacro:include filename="$(find youbot_description)/urdf/youbot_gripper/gripper.urdf.xacro" />
   <!-- generic simulator_gazebo plugins for starting mechanism control, ros time, ros battery -->
-  <include filename="$(find youbot_description)/gazebo/gazebo.urdf.xacro" />
+  <xacro:include filename="$(find youbot_description)/gazebo/gazebo.urdf.xacro" />
   <!-- materials for visualization -->
-  <include filename="$(find youbot_description)/urdf/materials.urdf.xacro" />
+  <xacro:include filename="$(find youbot_description)/urdf/materials.urdf.xacro" />
   <!-- Now we can start using the macros included above to define the actual youbot -->
   <!-- The first use of a macro.  This one was defined in base.urdf.xacro above.

File: workspaces/youbot/src/youbot_description/robots/youbot_gripper.urdf__OLD__.xacro (robot description, xacro)
@@ -7,11 +7,11 @@
   <!-- The following included files set up definitions of parts of the robot body -->
   <!-- misc common stuff? -->
-  <include filename="$(find youbot_description)/urdf/common.xacro" />
+  <xacro:include filename="$(find youbot_description)/urdf/common.xacro" />
   <!-- youbot gripper -->
-  <include filename="$(find youbot_description)/urdf/youbot_gripper/gripper.urdf.xacro" />
+  <xacro:include filename="$(find youbot_description)/urdf/youbot_gripper/gripper.urdf.xacro" />
   <!-- generic simulator_gazebo plugins for starting mechanism control, ros time, ros battery -->
-  <include filename="$(find youbot_description)/gazebo/gazebo.urdf.xacro" />
+  <xacro:include filename="$(find youbot_description)/gazebo/gazebo.urdf.xacro" />
   <!-- materials for visualization -->
-  <include filename="$(find youbot_description)/urdf/materials.urdf.xacro" />
+  <xacro:include filename="$(find youbot_description)/urdf/materials.urdf.xacro" />
   <!-- Now we can start using the macros included above to define the actual youbot -->
   <!-- The first use of a macro.  This one was defined in base.urdf.xacro above.

File: workspaces/youbot/src/youbot_description/urdf/sensors/asus_xtion_camera.urdf.xacro (robot description, xacro)
@@ -5,5 +5,5 @@
         xmlns:xacro="http://ros.org/wiki/xacro">
   <property name="M_PI" value="3.14159"/>.
-  <include filename="$(find youbot_description)/urdf/sensors/asus_xtion_camera.gazebo.xacro" />
+  <xacro:include filename="$(find youbot_description)/urdf/sensors/asus_xtion_camera.gazebo.xacro" />
   <property name="eye_x_offset" value="0.03" />
   <property name="eye_y_offset" value="0.035" />

File: workspaces/youbot/src/youbot_description/urdf/sensors/hokuyo_urg04_laser.urdf.xacro (robot description, xacro)
@@ -4,5 +4,5 @@
        xmlns:interface="http://playerstage.sourceforge.net/gazebo/xmlschema/#interface"
        xmlns:xacro="http://ros.org/wiki/xacro">
-  <include filename="$(find youbot_description)/urdf/sensors/hokuyo_urg04_laser.gazebo.xacro" />
+  <xacro:include filename="$(find youbot_description)/urdf/sensors/hokuyo_urg04_laser.gazebo.xacro" />
   <xacro:macro name="hokuyo_urg04_laser" params="name parent *origin ros_topic update_rate min_angle max_angle">
     <joint name="${name}_hokuyo_urg04_laser_joint" type="fixed">

File: workspaces/youbot/src/youbot_description/urdf/sensors/kinect_camera.urdf.xacro (robot description, xacro)
@@ -4,5 +4,5 @@
       xmlns:interface="http://playerstage.sourceforge.net/gazebo/xmlschema/#interface"
       xmlns:xacro="http://ros.org/wiki/xacro">
-  <include filename="$(find youbot_description)/urdf/sensors/kinect_camera.gazebo.xacro"/>
+  <xacro:include filename="$(find youbot_description)/urdf/sensors/kinect_camera.gazebo.xacro"/>
   <xacro:macro name="kinect_camera" params="name parent *origin">
    <joint name="${name}_camera_joint" type="fixed">

File: workspaces/youbot/src/youbot_description/urdf/sensors/microsoft_lifecam.urdf.xacro (robot description, xacro)
@@ -4,5 +4,5 @@
       xmlns:interface="http://playerstage.sourceforge.net/gazebo/xmlschema/#interface"
       xmlns:xacro="http://ros.org/wiki/xacro">
-  <include filename="$(find youbot_description)/urdf/sensors/microsoft_lifecam.gazebo.xacro"/>
+  <xacro:include filename="$(find youbot_description)/urdf/sensors/microsoft_lifecam.gazebo.xacro"/>
   <xacro:macro name="microsoft_lifecam" params="name parent *origin">
    <joint name="${name}_camera_joint" type="fixed">

File: workspaces/youbot/src/youbot_description/urdf/youbot_arm/arm.urdf.xacro (robot description, xacro)
@@ -4,7 +4,7 @@
         xmlns:interface="http://playerstage.sourceforge.net/gazebo/xmlschema/#interface"
         xmlns:xacro="http://ros.org/wiki/xacro">
-	<include filename="$(find youbot_description)/urdf/youbot_arm/arm.gazebo.xacro" />
-	<include filename="$(find youbot_description)/urdf/youbot_arm/arm.transmission.xacro" />
-        <include filename="$(find youbot_description)/urdf/youbot_arm/limits.urdf.xacro" />
+	<xacro:include filename="$(find youbot_description)/urdf/youbot_arm/arm.gazebo.xacro" />
+	<xacro:include filename="$(find youbot_description)/urdf/youbot_arm/arm.transmission.xacro" />
+        <xacro:include filename="$(find youbot_description)/urdf/youbot_arm/limits.urdf.xacro" />
 	<xacro:macro name="youbot_arm" params="parent name *origin">
 		<!-- joint between base_link and arm_0_link -->

File: workspaces/youbot/src/youbot_description/urdf/youbot_base/base.urdf.xacro (robot description, xacro)
@@ -5,7 +5,7 @@
         xmlns:xacro="http://ros.org/wiki/xacro">
 	<!-- sensors -->
-	<include filename="$(find youbot_description)/urdf/sensors/hokuyo_urg04_laser.urdf.xacro"/>
-	<include filename="$(find youbot_description)/urdf/youbot_base/base.gazebo.xacro" />
-	<include filename="$(find youbot_description)/urdf/youbot_base/base.transmission.xacro" />
+	<xacro:include filename="$(find youbot_description)/urdf/sensors/hokuyo_urg04_laser.urdf.xacro"/>
+	<xacro:include filename="$(find youbot_description)/urdf/youbot_base/base.gazebo.xacro" />
+	<xacro:include filename="$(find youbot_description)/urdf/youbot_base/base.transmission.xacro" />
  	<!-- simplified box collision geometry for base -->
   	<property name="base_size_x" value="0.570" />

File: workspaces/youbot/src/youbot_description/urdf/youbot_base/base.urdf__OLD__.xacro (robot description, xacro)
@@ -5,7 +5,7 @@
         xmlns:xacro="http://ros.org/wiki/xacro">
 	<!-- sensors -->
-	<include filename="$(find youbot_description)/urdf/sensors/hokuyo_urg04_laser.urdf.xacro"/>
-	<include filename="$(find youbot_description)/urdf/youbot_base/base.gazebo.xacro" />
-	<include filename="$(find youbot_description)/urdf/youbot_base/base.transmission.xacro" />
+	<xacro:include filename="$(find youbot_description)/urdf/sensors/hokuyo_urg04_laser.urdf.xacro"/>
+	<xacro:include filename="$(find youbot_description)/urdf/youbot_base/base.gazebo.xacro" />
+	<xacro:include filename="$(find youbot_description)/urdf/youbot_base/base.transmission.xacro" />
  	<!-- simplified box collision geometry for base -->
   	<property name="base_size_x" value="0.570" />

File: workspaces/youbot/src/youbot_description/urdf/youbot_gripper/gripper.urdf.xacro (robot description, xacro)
@@ -4,8 +4,8 @@
        xmlns:interface="http://playerstage.sourceforge.net/gazebo/xmlschema/#interface"
        xmlns:xacro="http://ros.org/wiki/xacro">
-	<include filename="$(find youbot_description)/urdf/youbot_gripper/gripper.gazebo.xacro" />
-	<include filename="$(find youbot_description)/urdf/youbot_gripper/gripper.transmission.xacro" />
-	<include filename="$(find youbot_description)/urdf/youbot_gripper/limits.urdf.xacro" />
-<!--	<include filename="$(find youbot_description)/urdf/sensors/asus_xtion_camera.urdf.xacro" /> -->
+	<xacro:include filename="$(find youbot_description)/urdf/youbot_gripper/gripper.gazebo.xacro" />
+	<xacro:include filename="$(find youbot_description)/urdf/youbot_gripper/gripper.transmission.xacro" />
+	<xacro:include filename="$(find youbot_description)/urdf/youbot_gripper/limits.urdf.xacro" />
+<!--	<xacro:include filename="$(find youbot_description)/urdf/sensors/asus_xtion_camera.urdf.xacro" /> -->
 	<xacro:macro name="youbot_gripper" params="parent name *origin">
 		<!-- joint between arm_link_5 and sdh_palm_link -->

File: workspaces/youbot/src/youbot_description/urdf/youbot_gripper/gripper.urdf__OLD__.xacro (robot description, xacro)
@@ -4,7 +4,7 @@
        xmlns:interface="http://playerstage.sourceforge.net/gazebo/xmlschema/#interface"
        xmlns:xacro="http://ros.org/wiki/xacro">
-	<include filename="$(find youbot_description)/urdf/youbot_gripper/gripper.gazebo.xacro" />
-	<include filename="$(find youbot_description)/urdf/youbot_gripper/gripper.transmission.xacro" />
-	<include filename="$(find youbot_description)/urdf/youbot_gripper/limits.urdf.xacro" />
+	<xacro:include filename="$(find youbot_description)/urdf/youbot_gripper/gripper.gazebo.xacro" />
+	<xacro:include filename="$(find youbot_description)/urdf/youbot_gripper/gripper.transmission.xacro" />
+	<xacro:include filename="$(find youbot_description)/urdf/youbot_gripper/limits.urdf.xacro" />
 	<xacro:macro name="youbot_gripper" params="parent name *origin">
 		<!-- joint between arm_7_link and sdh_palm_link -->
