Commit message: fixed the gripper position

File: workspaces/youbot/src/youbot_description/robots/youbot.urdf.xacro (robot description, xacro)
@@ -40,8 +40,8 @@
   <xacro:youbot_arm name="arm_2" parent="base_link">
     <!--<origin xyz="-0.143 0 0.046" rpy="0 0 3.1415" />-->
-    <origin xyz="-0.123 0 0.046" rpy="0 0 3.1415" />  <!-- x offset needs to be further verified -->
+    <origin xyz="-0.143 0 0.056" rpy="0 0 3.1415" />  <!-- x offset needs to be further verified -->
   </xacro:youbot_arm>
   <xacro:youbot_gripper name="gripper_2" parent="arm_2_link_5">
-    <origin xyz="0 0 0" rpy="0 0 0" />
+    <origin xyz="-0.0027 0 .016" rpy="0 ${-M_PI/2} ${M_PI}" />
   </xacro:youbot_gripper>
 <!-- SENSOR SPECIFIC STUFF -->

Commit message: one arm config

File: workspaces/youbot/src/youbot_description/robots/youbot.urdf.xacro (robot description, xacro)
@@ -37,12 +37,12 @@
     <origin xyz="-0.0027 0 .016" rpy="0 ${-M_PI/2} ${M_PI}" />
   </xacro:youbot_gripper>
-<!--Second arm-->
-  <xacro:youbot_arm name="arm_2" parent="base_link">
-    <!--<origin xyz="-0.143 0 0.046" rpy="0 0 3.1415" />-->
-    <origin xyz="-0.143 0 0.056" rpy="0 0 3.1415" />  <!-- x offset needs to be further verified -->
-  </xacro:youbot_arm>
-  <xacro:youbot_gripper name="gripper_2" parent="arm_2_link_5">
-    <origin xyz="-0.0027 0 .016" rpy="0 ${-M_PI/2} ${M_PI}" />
-  </xacro:youbot_gripper>
+<!--<!--Second arm-->-->
+<!--  <xacro:youbot_arm name="arm_2" parent="base_link">-->
+<!--    <!--<origin xyz="-0.143 0 0.046" rpy="0 0 3.1415" />-->-->
+<!--    <origin xyz="-0.143 0 0.056" rpy="0 0 3.1415" />  <!-- x offset needs to be further verified -->-->
+<!--  </xacro:youbot_arm>-->
+<!--  <xacro:youbot_gripper name="gripper_2" parent="arm_2_link_5">-->
+<!--    <origin xyz="-0.0027 0 .016" rpy="0 ${-M_PI/2} ${M_PI}" />-->
+<!--  </xacro:youbot_gripper>-->
 <!-- SENSOR SPECIFIC STUFF -->
   <include filename="$(find youbot_description)/urdf/updated_materials.urdf.xacro" />

Commit message: minor edit

File: workspaces/youbot/src/youbot_description/robots/youbot.urdf.xacro (robot description, xacro)
@@ -37,8 +37,8 @@
     <origin xyz="-0.0027 0 .016" rpy="0 ${-M_PI/2} ${M_PI}" />
   </xacro:youbot_gripper>
-<!--<!--Second arm-->-->
+<!--Second arm-->
 <!--  <xacro:youbot_arm name="arm_2" parent="base_link">-->
-<!--    <!--<origin xyz="-0.143 0 0.046" rpy="0 0 3.1415" />-->-->
-<!--    <origin xyz="-0.143 0 0.056" rpy="0 0 3.1415" />  <!-- x offset needs to be further verified -->-->
+        <!--<origin xyz="-0.143 0 0.046" rpy="0 0 3.1415" />-->
+<!--    <origin xyz="-0.143 0 0.056" rpy="0 0 3.1415" />  --> <!-- x offset needs to be further verified -->
 <!--  </xacro:youbot_arm>-->
 <!--  <xacro:youbot_gripper name="gripper_2" parent="arm_2_link_5">-->

Commit message: added 'invisible' 0; has no real effect, just cosmetic

File: workspaces/youbot/src/youbot_description/robots/youbot.urdf.xacro (robot description, xacro)
@@ -35,5 +35,5 @@
   </xacro:youbot_arm>
   <xacro:youbot_gripper name="gripper" parent="arm_link_5">
-    <origin xyz="-0.0027 0 .016" rpy="0 ${-M_PI/2} ${M_PI}" />
+    <origin xyz="-0.0027 0 0.016" rpy="0 ${-M_PI/2} ${M_PI}" />
   </xacro:youbot_gripper>
 <!--Second arm-->

Commit message: two arm config in urdf

File: workspaces/youbot/src/youbot_description/robots/youbot.urdf.xacro (robot description, xacro)
@@ -38,11 +38,11 @@
   </xacro:youbot_gripper>
 <!--Second arm-->
-<!--  <xacro:youbot_arm name="arm_2" parent="base_link">-->
+  <xacro:youbot_arm name="arm_2" parent="base_link">
         <!--<origin xyz="-0.143 0 0.046" rpy="0 0 3.1415" />-->
-<!--    <origin xyz="-0.143 0 0.056" rpy="0 0 3.1415" />  --> <!-- x offset needs to be further verified -->
-<!--  </xacro:youbot_arm>-->
-<!--  <xacro:youbot_gripper name="gripper_2" parent="arm_2_link_5">-->
-<!--    <origin xyz="-0.0027 0 .016" rpy="0 ${-M_PI/2} ${M_PI}" />-->
-<!--  </xacro:youbot_gripper>-->
+        <origin xyz="-0.143 0 0.056" rpy="0 0 3.1415" />   <!-- x offset needs to be further verified -->
+  </xacro:youbot_arm>
+  <xacro:youbot_gripper name="gripper_2" parent="arm_2_link_5">
+    <origin xyz="-0.0027 0 0.016" rpy="0 ${-M_PI/2} ${M_PI}" />
+  </xacro:youbot_gripper>
 <!-- SENSOR SPECIFIC STUFF -->
   <include filename="$(find youbot_description)/urdf/updated_materials.urdf.xacro" />

Commit message: replaced one arm with plate

File: workspaces/youbot/src/youbot_description/robots/youbot.urdf.xacro (robot description, xacro)
@@ -38,11 +38,16 @@
   </xacro:youbot_gripper>
 <!--Second arm-->
-  <xacro:youbot_arm name="arm_2" parent="base_link">
+<!-- <xacro:youbot_arm name="arm_2" parent="base_link"> -->
         <!--<origin xyz="-0.143 0 0.046" rpy="0 0 3.1415" />-->
-        <origin xyz="-0.143 0 0.056" rpy="0 0 3.1415" />   <!-- x offset needs to be further verified -->
-  </xacro:youbot_arm>
+<!--        <origin xyz="-0.143 0 0.056" rpy="0 0 3.1415" />  -->  <!-- x offset needs to be further verified -->
+<!--  </xacro:youbot_arm>
   <xacro:youbot_gripper name="gripper_2" parent="arm_2_link_5">
     <origin xyz="-0.0027 0 0.016" rpy="0 ${-M_PI/2} ${M_PI}" />
   </xacro:youbot_gripper>
+-->
+<!-- PLATE -->
+ <xacro:youbot_plate name="plate" parent="base_link">
+    <origin xyz="-0.159 0 0.055" rpy="0 0 0" />
+  </xacro:youbot_plate>
 <!-- SENSOR SPECIFIC STUFF -->
   <include filename="$(find youbot_description)/urdf/updated_materials.urdf.xacro" />

Commit message: added minor offset to camera pos

File: workspaces/youbot/src/youbot_description/robots/youbot.urdf.xacro (robot description, xacro)
@@ -70,5 +70,5 @@
   <xacro:asus_xtion_camera name="xtion" parent="arm_sensor_angle_part2_link"  tilt="0.0">
   <!-- AR_CALIBRATOR:EDIT_HERE -->
-    <origin xyz="0.01 0.0 0.0" rpy="${M_PI} 0.0 ${M_PI}" />
+    <origin xyz="0.00 0.0 0.01" rpy="${M_PI} 0.0 ${M_PI}" />
   </xacro:asus_xtion_camera>
 </robot>

Commit message: new calibration info

File: workspaces/youbot/src/youbot_description/robots/youbot.urdf.xacro (robot description, xacro)
@@ -70,5 +70,5 @@
   <xacro:asus_xtion_link name="xtion" parent="arm_sensor_angle_part2_link"  tilt="0.0">
   <!-- AR_CALIBRATOR:EDIT_HERE -->
-    <origin xyz="0.00 0.0 0.01" rpy="${M_PI} 0.0 ${M_PI}" />
+                  <origin xyz="-0.0257147 0.0282211 -0.0477212" rpy="3.13912 -0.275912 -3.12588" />
   </xacro:asus_xtion_link>
 </robot>

Commit message: updated calib values in urdf

File: workspaces/youbot/src/youbot_description/robots/youbot.urdf.xacro (robot description, xacro)
@@ -70,5 +70,5 @@
   <xacro:asus_xtion_link name="xtion" parent="arm_sensor_angle_part2_link"  tilt="0.0">
   <!-- AR_CALIBRATOR:EDIT_HERE -->
-                  <origin xyz="-0.0257147 0.0282211 -0.0477212" rpy="3.13912 -0.275912 -3.12588" />
+                  <origin xyz="-0.0256356 0.0275046 -0.0475053" rpy="3.14097 -0.273895 -3.1287" />
   </xacro:asus_xtion_link>
 </robot>

Commit message: Signed-off-by: yiming_yang <yymalex@gmail.com>

File: workspaces/youbot/src/youbot_description/robots/youbot.urdf.xacro (robot description, xacro)
@@ -7,17 +7,17 @@
   <!-- The following included files set up definitions of parts of the robot body -->
   <!-- misc common stuff? -->
-  <xacro:include filename="$(find youbot_description)/urdf/common.xacro" />
+  <include filename="$(find youbot_description)/urdf/common.xacro" />
   <!-- youbot base -->
-  <xacro:include filename="$(find youbot_description)/urdf/youbot_base/base.urdf.xacro" />
+  <include filename="$(find youbot_description)/urdf/youbot_base/base.urdf.xacro" />
   <!-- youbot plate -->
-  <xacro:include filename="$(find youbot_description)/urdf/youbot_plate/plate.urdf.xacro" />
+  <include filename="$(find youbot_description)/urdf/youbot_plate/plate.urdf.xacro" />
   <!-- youbot arm -->
-  <xacro:include filename="$(find youbot_description)/urdf/youbot_arm/arm.urdf.xacro"/>
+  <include filename="$(find youbot_description)/urdf/youbot_arm/arm.urdf.xacro"/>
   <!-- youbot gripper -->
-  <xacro:include filename="$(find youbot_description)/urdf/youbot_gripper/gripper.urdf.xacro" />
+  <include filename="$(find youbot_description)/urdf/youbot_gripper/gripper.urdf.xacro" />
   <!-- generic simulator_gazebo plugins for starting mechanism control, ros time, ros battery -->
-  <xacro:include filename="$(find youbot_description)/gazebo/gazebo.urdf.xacro" />
+  <include filename="$(find youbot_description)/gazebo/gazebo.urdf.xacro" />
   <!-- materials for visualization -->
-  <xacro:include filename="$(find youbot_description)/urdf/materials.urdf.xacro" />
+  <include filename="$(find youbot_description)/urdf/materials.urdf.xacro" />
   <!-- Now we can start using the macros included above to define the actual youbot -->
   <!-- The first use of a macro.  This one was defined in base.urdf.xacro above.
@@ -30,45 +30,12 @@
 <!-- foot for arm-->
   <xacro:youbot_base name="base"/>
-<!--First arm-->
+  <xacro:youbot_plate name="plate" parent="base_link">
+    <origin xyz="-0.159 0 0.046" rpy="0 0 0" />
+  </xacro:youbot_plate>
   <xacro:youbot_arm name="arm" parent="base_link">
-    <origin xyz="0.143 0 0.056" rpy="0 0 0" />
+    <origin xyz="0.143 0 0.046" rpy="0 0 0" />
   </xacro:youbot_arm>
   <xacro:youbot_gripper name="gripper" parent="arm_link_5">
-    <origin xyz="-0.0027 0 0.016" rpy="0 ${-M_PI/2} ${M_PI}" />
+    <origin xyz="0 0 0" rpy="0 0 0" />
   </xacro:youbot_gripper>
-<!--Second arm-->
-<!-- <xacro:youbot_arm name="arm_2" parent="base_link"> -->
-        <!--<origin xyz="-0.143 0 0.046" rpy="0 0 3.1415" />-->
-<!--        <origin xyz="-0.143 0 0.056" rpy="0 0 3.1415" />  -->  <!-- x offset needs to be further verified -->
-<!--  </xacro:youbot_arm>
-  <xacro:youbot_gripper name="gripper_2" parent="arm_2_link_5">
-    <origin xyz="-0.0027 0 0.016" rpy="0 ${-M_PI/2} ${M_PI}" />
-  </xacro:youbot_gripper>
--->
-<!-- PLATE -->
- <xacro:youbot_plate name="plate" parent="base_link">
-    <origin xyz="-0.159 0 0.055" rpy="0 0 0" />
-  </xacro:youbot_plate>
-<!-- SENSOR SPECIFIC STUFF -->
-  <xacro:include filename="$(find youbot_description)/urdf/updated_materials.urdf.xacro" />
-  <xacro:include filename="$(find youbot_description)/urdf/misc/sensor_angle.urdf.xacro" />
-<!--  <xacro:include filename="$(find youbot_description)/urdf/misc/cam3d_tower.urdf.xacro" /> -->
-<!--  <xacro:include filename="$(find youbot_description)/urdf/sensors/kinect_camera.urdf.xacro" /> -->
-<!--  <xacro:include filename="$(find youbot_description)/urdf/sensors/microsoft_lifecam.urdf.xacro" /> -->
-  <xacro:include filename="$(find youbot_description)/urdf/sensors/asus_xtion_camera.urdf.xacro" />
-  <!-- base laser rear -->
-<!--
-   <xacro:hokuyo_urg04_laser name="base_laser_rear" parent="base" ros_topic="scan_rear" update_rate="10" min_angle="-1.57" max_angle="1.57">
-     <origin xyz="-0.3 0.0 -0.03" rpy="0 0 ${M_PI}" />
-  </xacro:hokuyo_urg04_laser>
--->
-  <!-- Sensor angle on arm -->
-  <xacro:sensor_angle name="arm_sensor_angle" parent="arm_link_5">
-    <origin xyz="-0.002 0.0 -0.023" rpy="0.0 0.0 0.0" />
-  </xacro:sensor_angle>
-  <!-- ASUS Xtion on arm sensor angle -->
-  <xacro:asus_xtion_link name="xtion" parent="arm_sensor_angle_part2_link"  tilt="0.0">
-  <!-- AR_CALIBRATOR:EDIT_HERE -->
-                  <origin xyz="-0.0253595 0.0305853 -0.0469736" rpy="3.13948 -0.306551 -3.13083" />
-  </xacro:asus_xtion_link>
 </robot>

File: workspaces/youbot/src/youbot_description/robots/youbot_arm.urdf (copy).xacro (robot description, xacro)
@@ -8,10 +8,12 @@
   <!-- misc common stuff? -->
   <xacro:include filename="$(find youbot_description)/urdf/common.xacro" />
-  <!-- youbot gripper -->
+  <!-- materials for visualization -->
+  <xacro:include filename="$(find youbot_description)/urdf/materials.urdf.xacro" />
+  <!-- youbot arm -->
+  <xacro:include filename="$(find youbot_description)/urdf/youbot_arm/arm.urdf.xacro" />
+  <!-- youbot arm -->
   <xacro:include filename="$(find youbot_description)/urdf/youbot_gripper/gripper.urdf.xacro" />
   <!-- generic simulator_gazebo plugins for starting mechanism control, ros time, ros battery -->
   <xacro:include filename="$(find youbot_description)/gazebo/gazebo.urdf.xacro" />
-  <!-- materials for visualization -->
-  <xacro:include filename="$(find youbot_description)/urdf/materials.urdf.xacro" />
   <!-- Now we can start using the macros included above to define the actual youbot -->
   <!-- The first use of a macro.  This one was defined in base.urdf.xacro above.
@@ -24,6 +26,17 @@
 <!-- foot for arm-->
   <link name="base_link">
-  </link>
-  <xacro:youbot_gripper name="gripper" parent="base_link">
+    <inertial>
+		   <origin xyz="0 0 0" rpy="0 0 0"/>
+		   <mass value="10.0"/>
+		   <inertia ixx="0.1"  ixy="0"  ixz="0" iyy="0.1" iyz="0" izz="0.1" />
+    </inertial>
+    </link>
+    <gazebo reference="base_link">
+		   <material>youbot/Orange</material>
+    </gazebo>
+  <xacro:youbot_arm name="arm" parent="base_link">
+    <origin xyz="0 0 0" rpy="0 0 0" />
+  </xacro:youbot_arm>
+  <xacro:youbot_gripper name="gripper" parent="arm_link_5">
     <origin xyz="0 0 0" rpy="0 0 0" />
   </xacro:youbot_gripper>

File: workspaces/youbot/src/youbot_description/robots/youbot_arm.urdf.xacro (robot description, xacro)
@@ -32,7 +32,4 @@
     </inertial>
     </link>
-    <gazebo reference="base_link">
-		   <material>youbot/Orange</material>
-    </gazebo>
   <xacro:youbot_arm name="arm" parent="base_link">
     <origin xyz="0 0 0" rpy="0 0 0" />

File: workspaces/youbot/src/youbot_description/robots/youbot_gripper.urdf (copy).xacro (robot description, xacro)
@@ -8,12 +8,10 @@
   <!-- misc common stuff? -->
   <xacro:include filename="$(find youbot_description)/urdf/common.xacro" />
-  <!-- materials for visualization -->
-  <xacro:include filename="$(find youbot_description)/urdf/materials.urdf.xacro" />
-  <!-- youbot arm -->
-  <xacro:include filename="$(find youbot_description)/urdf/youbot_arm/arm.urdf.xacro" />
-  <!-- youbot arm -->
+  <!-- youbot gripper -->
   <xacro:include filename="$(find youbot_description)/urdf/youbot_gripper/gripper.urdf.xacro" />
   <!-- generic simulator_gazebo plugins for starting mechanism control, ros time, ros battery -->
   <xacro:include filename="$(find youbot_description)/gazebo/gazebo.urdf.xacro" />
+  <!-- materials for visualization -->
+  <xacro:include filename="$(find youbot_description)/urdf/materials.urdf.xacro" />
   <!-- Now we can start using the macros included above to define the actual youbot -->
   <!-- The first use of a macro.  This one was defined in base.urdf.xacro above.
@@ -26,14 +24,9 @@
 <!-- foot for arm-->
   <link name="base_link">
-    <inertial>
-		   <origin xyz="0 0 0" rpy="0 0 0"/>
-		   <mass value="10.0"/>
-		   <inertia ixx="0.1"  ixy="0"  ixz="0" iyy="0.1" iyz="0" izz="0.1" />
-    </inertial>
-    </link>
-  <xacro:youbot_arm name="arm" parent="base_link">
-    <origin xyz="0 0 0" rpy="0 0 0" />
-  </xacro:youbot_arm>
-  <xacro:youbot_gripper name="gripper" parent="arm_link_5">
+  </link>
+  <gazebo reference="base_link">
+       <material>youbot/DarkGrey</material>
+  </gazebo>
+  <xacro:youbot_gripper name="gripper" parent="base_link">
     <origin xyz="0 0 0" rpy="0 0 0" />
   </xacro:youbot_gripper>

File: workspaces/youbot/src/youbot_description/robots/youbot_gripper.urdf.xacro (robot description, xacro)
@@ -25,7 +25,4 @@
   <link name="base_link">
   </link>
-  <gazebo reference="base_link">
-       <material>youbot/DarkGrey</material>
-  </gazebo>
   <xacro:youbot_gripper name="gripper" parent="base_link">
     <origin xyz="0 0 0" rpy="0 0 0" />
