Commit message: Functional detection and planning. Detecting, locating target. Generating IK for gripper to target pose. Planning, moving. Signed-off-by: yiming <yymalex@gmail.com>

File: workspaces/youbot/src/youbot_description/robots/youbot.urdf.xacro (robot description, xacro)
@@ -7,17 +7,17 @@
   <!-- The following included files set up definitions of parts of the robot body -->
   <!-- misc common stuff? -->
-  <include filename="$(find youbot_description)/urdf/common.xacro" />
+  <xacro:include filename="$(find youbot_description)/urdf/common.xacro" />
   <!-- youbot base -->
-  <include filename="$(find youbot_description)/urdf/youbot_base/base.urdf.xacro" />
+  <xacro:include filename="$(find youbot_description)/urdf/youbot_base/base.urdf.xacro" />
   <!-- youbot plate -->
-  <include filename="$(find youbot_description)/urdf/youbot_plate/plate.urdf.xacro" />
+  <xacro:include filename="$(find youbot_description)/urdf/youbot_plate/plate.urdf.xacro" />
   <!-- youbot arm -->
-  <include filename="$(find youbot_description)/urdf/youbot_arm/arm.urdf.xacro"/>
+  <xacro:include filename="$(find youbot_description)/urdf/youbot_arm/arm.urdf.xacro"/>
   <!-- youbot gripper -->
-  <include filename="$(find youbot_description)/urdf/youbot_gripper/gripper.urdf.xacro" />
+  <xacro:include filename="$(find youbot_description)/urdf/youbot_gripper/gripper.urdf.xacro" />
   <!-- generic simulator_gazebo plugins for starting mechanism control, ros time, ros battery -->
-  <include filename="$(find youbot_description)/gazebo/gazebo.urdf.xacro" />
+  <xacro:include filename="$(find youbot_description)/gazebo/gazebo.urdf.xacro" />
   <!-- materials for visualization -->
-  <include filename="$(find youbot_description)/urdf/materials.urdf.xacro" />
+  <xacro:include filename="$(find youbot_description)/urdf/materials.urdf.xacro" />
   <!-- Now we can start using the macros included above to define the actual youbot -->
   <!-- The first use of a macro.  This one was defined in base.urdf.xacro above.
@@ -30,12 +30,45 @@
 <!-- foot for arm-->
   <xacro:youbot_base name="base"/>
-  <xacro:youbot_plate name="plate" parent="base_link">
-    <origin xyz="-0.159 0 0.046" rpy="0 0 0" />
-  </xacro:youbot_plate>
+<!--First arm-->
   <xacro:youbot_arm name="arm" parent="base_link">
-    <origin xyz="0.143 0 0.046" rpy="0 0 0" />
+    <origin xyz="0.143 0 0.056" rpy="0 0 0" />
   </xacro:youbot_arm>
   <xacro:youbot_gripper name="gripper" parent="arm_link_5">
-    <origin xyz="0 0 0" rpy="0 0 0" />
+    <origin xyz="-0.0027 0 0.016" rpy="0 ${-M_PI/2} ${M_PI}" />
   </xacro:youbot_gripper>
+<!--Second arm-->
+<!-- <xacro:youbot_arm name="arm_2" parent="base_link"> -->
+        <!--<origin xyz="-0.143 0 0.046" rpy="0 0 3.1415" />-->
+<!--        <origin xyz="-0.143 0 0.056" rpy="0 0 3.1415" />  -->  <!-- x offset needs to be further verified -->
+<!--  </xacro:youbot_arm>
+  <xacro:youbot_gripper name="gripper_2" parent="arm_2_link_5">
+    <origin xyz="-0.0027 0 0.016" rpy="0 ${-M_PI/2} ${M_PI}" />
+  </xacro:youbot_gripper>
+-->
+<!-- PLATE -->
+ <xacro:youbot_plate name="plate" parent="base_link">
+    <origin xyz="-0.159 0 0.055" rpy="0 0 0" />
+  </xacro:youbot_plate>
+<!-- SENSOR SPECIFIC STUFF -->
+  <xacro:include filename="$(find youbot_description)/urdf/updated_materials.urdf.xacro" />
+  <xacro:include filename="$(find youbot_description)/urdf/misc/sensor_angle.urdf.xacro" />
+<!--  <xacro:include filename="$(find youbot_description)/urdf/misc/cam3d_tower.urdf.xacro" /> -->
+<!--  <xacro:include filename="$(find youbot_description)/urdf/sensors/kinect_camera.urdf.xacro" /> -->
+<!--  <xacro:include filename="$(find youbot_description)/urdf/sensors/microsoft_lifecam.urdf.xacro" /> -->
+  <xacro:include filename="$(find youbot_description)/urdf/sensors/asus_xtion_camera.urdf.xacro" />
+  <!-- base laser rear -->
+<!--
+   <xacro:hokuyo_urg04_laser name="base_laser_rear" parent="base" ros_topic="scan_rear" update_rate="10" min_angle="-1.57" max_angle="1.57">
+     <origin xyz="-0.3 0.0 -0.03" rpy="0 0 ${M_PI}" />
+  </xacro:hokuyo_urg04_laser>
+-->
+  <!-- Sensor angle on arm -->
+  <xacro:sensor_angle name="arm_sensor_angle" parent="arm_link_5">
+    <origin xyz="-0.002 0.0 -0.023" rpy="0.0 0.0 0.0" />
+  </xacro:sensor_angle>
+  <!-- ASUS Xtion on arm sensor angle -->
+  <xacro:asus_xtion_link name="xtion" parent="arm_sensor_angle_part2_link"  tilt="0.0">
+  <!-- AR_CALIBRATOR:EDIT_HERE -->
+                  <origin xyz="-0.0210658 0.0348332 -0.037004" rpy="3.12964 -0.00987025 -3.13267" />
+  </xacro:asus_xtion_link>
 </robot>

File: workspaces/youbot/src/youbot_description/robots/youbot_baseIK.urdf.xacro (robot description, xacro)
@@ -70,5 +70,5 @@
   <xacro:asus_xtion_link name="xtion" parent="arm_sensor_angle_part2_link"  tilt="0.0">
   <!-- AR_CALIBRATOR:EDIT_HERE -->
-                  <origin xyz="-0.0253595 0.0305853 -0.0469736" rpy="3.13948 -0.306551 -3.13083" />
+                  <origin xyz="-0.0210658 0.0348332 -0.037004" rpy="3.12964 -0.00987025 -3.13267" />
   </xacro:asus_xtion_link>
 </robot>

File: workspaces/youbot/src/youbot_description/urdf/youbot_base/base_within_IK.urdf.xacro (robot description, xacro)
@@ -35,5 +35,5 @@
 	<xacro:macro name="youbot_base" params="name">
 		<link name="${name}_footprint">
-      			<inertial>
+      			<!--inertial>
         			<mass value="0.0001" />
         			<origin xyz="0 0 ${-base_size_z / 2.0}" rpy="0 0 0" />
@@ -53,38 +53,6 @@
           				<box size="0.001 0.001 0.001" />
         			</geometry>
-      			</collision>
-    		</link>
-		<link name="base_dummy_prismatic_x_link">
-		</link>
-		<link name="base_dummy_prismatic_y_link">
-		</link>
-		<link name="base_dummy_revolute_link">
-		</link>
-		<joint name="${name}_footprint_joint" type="fixed">
-      			<origin xyz="0 0 0" rpy="0 0 0" />
-      			<child link="base_dummy_revolute_link" />
-      			<parent link="${name}_footprint"/>
-    		</joint>
-		<joint name="base_dummy_revolute_joint" type="revolute">
-      			<origin xyz="0 0 0" rpy="0 0 0" />
-			<axis xyz="0 0 1" />
-			<child link="base_dummy_prismatic_x_link" />
-      			<parent link="base_dummy_revolute_link"/>
-			<limit effort="${9.5}" velocity="${M_PI}" lower="${-M_PI}" upper="${M_PI}"/>
-    		</joint>
-		<joint name="base_dummy_prismatic_x_joint" type="prismatic">
-      			<origin xyz="0 0 0" rpy="0 0 0" />
-			<axis xyz="1 0 0" />
-			<child link="base_dummy_prismatic_y_link" />
-      			<parent link="base_dummy_prismatic_x_link"/>
-			<limit effort="${9.5}" velocity="${M_PI}" lower="${-50}" upper="${50}"/>
-    		</joint>
-		<joint name="base_dummy_prismatic_y_joint" type="prismatic">
-      			<origin xyz="0 0 0" rpy="0 0 0" />
-			<axis xyz="0 1 0" />
-			<child link="${name}_link" />
-      			<parent link="base_dummy_prismatic_y_link"/>
-			<limit effort="${9.5}" velocity="${M_PI}" lower="${-50}" upper="${50}"/>
-    		</joint>
+      			</collision-->
+    		</link>
 		<link name="${name}_link">
       			<inertial>
@@ -109,4 +77,67 @@
       			</collision>
     		</link>
+		<link name="dummy_prismatic_link">
+			<inertial>
+        			<mass value="0.0001" />
+        			<origin xyz="0 0 ${-base_size_z / 2.0}" rpy="0 0 0" />
+        			<inertia ixx="1.0" ixy="0.0" ixz="0.0"
+                 			iyy="1.0" iyz="0.0" izz="1.0" />
+      				</inertial>
+      			<visual>
+        			<origin xyz="0 0 0" rpy="0 0 0" />
+        			<geometry>
+          				<box size="0.001 0.001 0.001" />
+        			</geometry>
+               			<material name="Red" />
+      			</visual>
+      			<collision>
+        			<origin xyz="0 0 ${-base_size_z / 2.0}" rpy="0 0 0" />
+        			<geometry>
+          				<box size="0.001 0.001 0.001" />
+        			</geometry>
+      			</collision>
+		</link>
+		<link name="dummy_revolute_link">
+			<inertial>
+        			<mass value="0.0001" />
+        			<origin xyz="0 0 ${-base_size_z / 2.0}" rpy="0 0 0" />
+        			<inertia ixx="1.0" ixy="0.0" ixz="0.0"
+                 			iyy="1.0" iyz="0.0" izz="1.0" />
+      				</inertial>
+      			<visual>
+        			<origin xyz="0 0 0" rpy="0 0 0" />
+        			<geometry>
+          				<box size="0.001 0.001 0.001" />
+        			</geometry>
+               			<material name="Red" />
+      			</visual>
+      			<collision>
+        			<origin xyz="0 0 ${-base_size_z / 2.0}" rpy="0 0 0" />
+        			<geometry>
+          				<box size="0.001 0.001 0.001" />
+        			</geometry>
+      			</collision>
+		</link>
+		<joint name="dummy_prismatic_x_joint" type="prismatic">
+			<origin xyz="0 0 0" rpy="0 0 0" />
+			<axis xyz="1 0 0" />
+			<limit effort="${9.5}" velocity="${M_PI}" lower="${-50}" upper="${50}"/>
+      			<child link="dummy_prismatic_link" />
+      			<parent link="${name}_footprint"/>
+    		</joint>
+		<joint name="dummy_prismatic_y_joint" type="prismatic">
+      			<origin xyz="0 0 0" rpy="0 0 0" />
+			<axis xyz="0 1 0" />
+			<child link="dummy_revolute_link" />
+      			<parent link="dummy_prismatic_link"/>
+			<limit effort="${9.5}" velocity="${M_PI}" lower="${-50}" upper="${50}"/>
+    		</joint>
+		<joint name="dummy_revolute_joint" type="revolute">
+      			<origin xyz="0 0 0" rpy="0 0 0" />
+			<axis xyz="0 0 1" />
+			<child link="${name}_link" />
+      			<parent link="dummy_revolute_link"/>
+			<limit effort="${9.5}" velocity="${M_PI}" lower="${-M_PI}" upper="${M_PI}"/>
+    		</joint>
 		<!-- base laser front -->
     		<xacro:hokuyo_urg04_laser name="${name}_laser_front" parent="${name}" ros_topic="scan_front" update_rate="10" min_angle="-1.57" max_angle="1.57" >
