Commit message: changed the urdf to match actual config, changed launch files accordingly, added an openni launcher for the xtion sensor

File: workspaces/youbot/src/youbot_description/robots/youbot.urdf (robot description, URDF)
Before this commit: robot youbot, 23 links, 22 joints
Links:
- removed link gripper_camera_collision_box_link
- added link arm_sensor_angle_part1_link, mass 0.01; collision box size=0.0625 0.097 0.0015; visual box size=0.0625 0.097 0.0015
- added link arm_sensor_angle_part2_link, mass 0.01; collision box size=0.0625 0.097 0.0015; visual box size=0.0625 0.097 0.0015
- added link base_laser_rear_link, mass 0.16; collision mesh filename=package://youbot_description/meshes/sensors/hokuyo_convex.d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; visual mesh filename=package://youbot_description/meshes/sensors/hokuyo.dae
- added link xtion_camera, mass 0.1; collision box size=0.2 0.06 0.07; visual mesh filename=package://youbot_description/meshes/sensors/asus_xtion_pro_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 scale=0.001 0.001 0.001
- added link xtion_depth_frame, mass 0.01
- added link xtion_depth_optical_frame, mass 0.01
- added link xtion_laser_frame, mass 0.01
- added link xtion_laser_optical_frame, mass 0.01
- added link xtion_rgb_frame, mass 0.01
- added link xtion_rgb_optical_frame, mass 0.01
- link arm_link_1: geometry collision mesh filename=package://youbot_description/meshes/youbot_arm/arm_joint_1_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; visual mesh filename=package://youbot_description/meshes/youbot_arm/arm1.dae
- link arm_link_2: geometry collision mesh filename=package://youbot_description/meshes/youbot_arm/arm_joint_2_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; visual mesh filename=package://youbot_description/meshes/youbot_arm/arm2.dae
- link arm_link_3: geometry collision mesh filename=package://youbot_description/meshes/youbot_arm/arm_joint_3_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; visual mesh filename=package://youbot_description/meshes/youbot_arm/arm3.dae
- link arm_link_4: geometry collision mesh filename=package://youbot_description/meshes/youbot_arm/arm_joint_4_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; visual mesh filename=package://youbot_description/meshes/youbot_arm/arm4.dae
- link arm_link_5: geometry collision mesh filename=package://youbot_description/meshes/youbot_arm/arm_joint_5_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; visual mesh filename=package://youbot_description/meshes/youbot_arm/arm5.dae
- link wheel_link_bl: geometry collision cylinder length=0.05 radius=0.05; visual mesh filename=package://youbot_description/meshes/youbot_base/back-left_w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
- link wheel_link_br: geometry collision cylinder length=0.05 radius=0.05; visual mesh filename=package://youbot_description/meshes/youbot_base/back-right_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
- link wheel_link_fl: geometry collision cylinder length=0.05 radius=0.05; visual mesh filename=package://youbot_description/meshes/youbot_base/front-left_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
- link wheel_link_fr: geometry collision cylinder length=0.05 radius=0.05; visual mesh filename=package://youbot_description/meshes/youbot_base/front-right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
Joints:
- removed joint gripper_camera_collision_box_joint
- added joint arm_sensor_angle_part1_joint: type fixed, parent arm_link_5, child arm_sensor_angle_part1_link, origin xyz=-0.002 0.0 -0.023 rpy=0.0 0.0 0.0
- added joint arm_sensor_angle_part2_joint: type fixed, parent arm_sensor_angle_part1_link, child arm_sensor_angle_part2_link, origin xyz=-0.0305 0 0.0305 rpy=0 1.570795 0 
- added joint arm_sensor_angle_part2_link_xtion_joint: type fixed, parent arm_sensor_angle_part2_link, child xtion_camera, origin xyz=0.01 0.0 0.0 rpy=3.14159 0.0 3.14159
- added joint base_laser_rear_hokuyo_urg04_laser_joint: type fixed, parent base_link, child base_laser_rear_link, origin xyz=-0.3 0.0 -0.03 rpy=0 0 3.14159, axis 0 1 0
- added joint xtion_depth_joint: type fixed, parent xtion_camera, child xtion_depth_frame, origin xyz=0.03 0.015 0 rpy=0 0 0
- added joint xtion_depth_optical_joint: type fixed, parent xtion_camera, child xtion_depth_optical_frame, origin xyz=0.03 0.015 0 rpy=-1.570795 0 -1.570795
- added joint xtion_laser_joint: type fixed, parent xtion_camera, child xtion_laser_frame, origin xyz=0.03 -0.055 0 rpy=0 0 0
- added joint xtion_laser_optical_joint: type fixed, parent xtion_camera, child xtion_laser_optical_frame, origin xyz=0.03 -0.055 0 rpy=1.570795 0 -1.570795
- added joint xtion_rgb_joint: type fixed, parent xtion_camera, child xtion_rgb_frame, origin xyz=0.03 -0.005 0 rpy=0 0 0
- added joint xtion_rgb_optical_joint: type fixed, parent xtion_camera, child xtion_rgb_optical_frame, origin xyz=0.03 -0.005 0 rpy=-1.570795 0 -1.570795
- joint arm_joint_0: origin xyz=0.143 0 0.046 rpy=0 0 0 -> xyz=0.143 0 0.056 rpy=0 0 0
- joint arm_joint_1: axis 0 0 1 -> 0 0 -1; limit lower=0 upper=5.89921287174 effort=9.5 velocity=1.57079632679 -> lower=0 upper=5.89920788889 effort=9.5 velocity=1.570795; origin xyz=0.024 0 0.115 rpy=0 0 -2.96705972839 -> xyz=0.024 0 0.115 rpy=0 0 2.96705722222
- joint arm_joint_2: axis 0 0 1 -> 0 1 0; limit lower=0 upper=2.70526034059 effort=9.5 velocity=1.57079632679 -> lower=0 upper=2.70525805556 effort=9.5 velocity=1.570795; origin xyz=0.033 0 0 rpy=-1.57079632679 0 1.57079632679 -> xyz=0.033 0 0 rpy=0 -1.13446305556 0
- joint arm_joint_3: limit lower=-5.18362787842 upper=0 effort=6.0 velocity=1.57079632679 -> lower=-5.1836235 upper=0 effort=6.0 velocity=1.570795; origin xyz=0.000 0.000 0.155 rpy=0 2.54818070791 0 -> xyz=0.000 0.000 0.155 rpy=0 2.54817855556 0
- joint arm_joint_4: limit lower=0 upper=3.57792496659 effort=2.0 velocity=1.57079632679 -> lower=0 upper=3.57792194444 effort=2.0 velocity=1.570795; origin xyz=0.000 0.000 0.135 rpy=0 -1.78896248329 0 -> xyz=0.000 0.000 0.135 rpy=0 -1.78896097222 0
- joint arm_joint_5: limit lower=0 upper=5.84685299418 effort=1 velocity=1.57079632679 -> lower=0 upper=5.84684805556 effort=1 velocity=1.570795; origin xyz=-0.002 0 0.130 rpy=0 0 2.92342649709 -> xyz=0 0 0.114 rpy=0 0 2.92342402778
- joint gripper_finger_joint_l: origin xyz=0.004 0.008 0.046 rpy=0 0 3.14159265359 -> xyz=0.046 0.010 0.003  rpy=0 -1.570795 3.14159
- joint gripper_finger_joint_r: origin xyz=0.004 -0.008 0.046 rpy=0 0 0 -> xyz=0.046 -0.010 0.003 rpy=0 1.570795 0
- joint gripper_palm_joint: origin xyz=0 0 0 rpy=0 0 0 -> xyz=-0.0027 0 .016 rpy=0 -1.570795 3.14159
- joint plate_joint: origin xyz=-0.159 0 0.046 rpy=0 0 0 -> xyz=-0.159 0 0.055 rpy=0 0 0

File: workspaces/youbot/src/youbot_description/robots/youbot.urdf.xacro (robot description, xacro)
@@ -30,7 +30,5 @@
 <!-- foot for arm-->
   <xacro:youbot_base name="base"/>
-  <xacro:youbot_plate name="plate" parent="base_link">
-    <origin xyz="-0.159 0 0.055" rpy="0 0 0" />
-  </xacro:youbot_plate>
+<!--First arm-->
   <xacro:youbot_arm name="arm" parent="base_link">
     <origin xyz="0.143 0 0.056" rpy="0 0 0" />
@@ -39,3 +37,30 @@
     <origin xyz="-0.0027 0 .016" rpy="0 ${-M_PI/2} ${M_PI}" />
   </xacro:youbot_gripper>
+<!--Second arm-->
+  <xacro:youbot_arm name="arm_2" parent="base_link">
+    <!--<origin xyz="-0.143 0 0.046" rpy="0 0 3.1415" />-->
+    <origin xyz="-0.123 0 0.046" rpy="0 0 3.1415" />  <!-- x offset needs to be further verified -->
+  </xacro:youbot_arm>
+  <xacro:youbot_gripper name="gripper_2" parent="arm_2_link_5">
+    <origin xyz="0 0 0" rpy="0 0 0" />
+  </xacro:youbot_gripper>
+<!-- SENSOR SPECIFIC STUFF -->
+  <include filename="$(find youbot_description)/urdf/updated_materials.urdf.xacro" />
+  <include filename="$(find youbot_description)/urdf/misc/sensor_angle.urdf.xacro" />
+<!--  <include filename="$(find youbot_description)/urdf/misc/cam3d_tower.urdf.xacro" /> -->
+<!--  <include filename="$(find youbot_description)/urdf/sensors/kinect_camera.urdf.xacro" /> -->
+<!--  <include filename="$(find youbot_description)/urdf/sensors/microsoft_lifecam.urdf.xacro" /> -->
+  <include filename="$(find youbot_description)/urdf/sensors/asus_xtion_camera.urdf.xacro" />
+  <!-- base laser rear -->
+  <xacro:hokuyo_urg04_laser name="base_laser_rear" parent="base" ros_topic="scan_rear" update_rate="10" min_angle="-1.57" max_angle="1.57">
+     <origin xyz="-0.3 0.0 -0.03" rpy="0 0 ${M_PI}" />
+  </xacro:hokuyo_urg04_laser>
+  <!-- Sensor angle on arm -->
+  <xacro:sensor_angle name="arm_sensor_angle" parent="arm_link_5">
+    <origin xyz="-0.002 0.0 -0.023" rpy="0.0 0.0 0.0" />
+  </xacro:sensor_angle>
+  <!-- ASUS Xtion on arm sensor angle -->
+  <xacro:asus_xtion_camera name="xtion" parent="arm_sensor_angle_part2_link"  tilt="0.0">
+    <origin xyz="0.01 0.0 0.0" rpy="${M_PI} 0.0 ${M_PI}" />
+  </xacro:asus_xtion_camera>
 </robot>

File: workspaces/youbot/src/youbot_description/urdf/youbot_gripper/gripper.urdf.xacro (robot description, xacro)
@@ -7,5 +7,5 @@
 	<include filename="$(find youbot_description)/urdf/youbot_gripper/gripper.transmission.xacro" />
 	<include filename="$(find youbot_description)/urdf/youbot_gripper/limits.urdf.xacro" />
-	<include filename="$(find youbot_description)/urdf/sensors/asus_xtion_camera.urdf.xacro" />
+<!--	<include filename="$(find youbot_description)/urdf/sensors/asus_xtion_camera.urdf.xacro" /> -->
 	<xacro:macro name="youbot_gripper" params="parent name *origin">
 		<!-- joint between arm_link_5 and sdh_palm_link -->
@@ -124,8 +124,8 @@
 		</gazebo>
                 <!-- asus xtion camera -->
-		<xacro:asus_xtion_camera name="xtion" parent="${name}_palm_link" tilt="0.0">
+<!--		<xacro:asus_xtion_camera name="xtion" parent="${name}_palm_link" tilt="0.0"> -->
                   <!-- AR_CALIBRATOR:EDIT_HERE -->
-                  <origin xyz="0.0197188 -0.0341838 0.0459352" rpy="0.0201114 0.00763208 3.0937" />
-                </xacro:asus_xtion_camera>
+<!--                  <origin xyz="0.0197188 -0.0341838 0.0459352" rpy="0.0201114 0.00763208 3.0937" />  -->
+<!--                </xacro:asus_xtion_camera>  -->
 		<!-- extensions -->
 		<xacro:youbot_gripper_gazebo name="${name}" />

Commit message: Signed-off-by: yiming <yymalex@gmail.com>

File: workspaces/youbot/src/youbot_description/robots/youbot.urdf (robot description, URDF)
Before this commit: robot youbot, 32 links, 31 joints
Links:
- added link dummy_prismatic_link
- added link dummy_revolute_link
- added link moveit_fixed_link
- link base_footprint: mass 0.0001 -> None; geometry 
- link base_link: geometry collision box size=0.57 0.36 0.1; visual mesh filename=package://youbot_description/meshes/youbot_base/base.dae
Joints:
- removed joint base_footprint_joint
- added joint dummy_prismatic_x_joint: type prismatic, parent moveit_fixed_link, child dummy_prismatic_link, origin xyz=0 0 0 rpy=0 0 0, axis 1 0 0, limit lower=-10.0 upper=10.0 effort=9.5 velocity=3.14159
- added joint dummy_prismatic_y_joint: type prismatic, parent dummy_prismatic_link, child dummy_revolute_link, origin xyz=0 0 0 rpy=0 0 0, axis 0 1 0, limit lower=-10.0 upper=10.0 effort=9.5 velocity=3.14159
- added joint dummy_revolute_joint: type revolute, parent dummy_revolute_link, child base_link, origin xyz=0 0 0 rpy=0 0 0, axis 0 0 1, limit lower=-3.14159 upper=3.14159 effort=9.5 velocity=3.14159
- added joint moveit_fixed_joint: type fixed, parent base_footprint, child moveit_fixed_link, origin xyz=0 0 0 rpy=0 0 0
