Commit message: added youbot descrption changes..

File: workspaces/youbot/src/youbot_description/urdf/youbot_arm/arm.urdf.xacro (robot description, xacro)
@@ -42,5 +42,6 @@
 		<!-- joint between arm_0_link and arm_1_link -->
 		<joint name="${name}_joint_1" type="revolute">
-			<origin xyz="0.024 0 0.115" rpy="0 0 ${170 * M_PI / 180}"/>
+			 <origin xyz="0.024 0 0.115" rpy="0 0 ${169 * M_PI / 180}"/>
+<!-- 			<origin xyz="0.024 0 0.115" rpy="0 0 0"/> -->
 			<parent link="${name}_link_0"/>
 			<child link="${name}_link_1"/>
@@ -50,5 +51,5 @@
 			<!-- damping - N*s/m, N*s*m/rad -->
 			<!-- friction - N, N*m -->
-			<limit effort="${9.5}" velocity="${M_PI / 2.0}" lower="0" upper="${joint_1_limit}"/>
+			<limit effort="${9.5}" velocity="${M_PI / 2.0}" lower="${0}" upper="${joint_1_limit}"/>
 			<!--effort - N, N*m-->
 			<!--velocity - m/s, rad/s-->
@@ -84,5 +85,6 @@
 		<!-- joint between arm_1_link and arm_2_link -->
 		<joint name="${name}_joint_2" type="revolute">
-			<origin xyz="0.033 0 0" rpy="0 ${-65 * M_PI / 180} 0"/>
+<!-- 			<origin xyz="0.033 0 0" rpy="0 ${-65 * M_PI / 180} 0"/> -->
+			<origin xyz="0.033 0 0" rpy="0 ${0 * M_PI / 180} 0"/>
 			<parent link="${name}_link_1"/>
 			<child link="${name}_link_2"/>
@@ -90,5 +92,5 @@
 			<!--<calibration rising="${arm_2_ref}" falling="${arm_2_ref}"/>-->
 			<dynamics damping="1" friction="1" />
-			<limit effort="${9.5}" velocity="${M_PI / 2.0}" lower="0" upper="${joint_2_limit}"/>
+			<limit effort="${9.5}" velocity="${M_PI / 2.0}" lower="-${joint_2_limit_low}" upper="${joint_2_limit_high}"/>
                         <safety_controller k_position="20" k_velocity="${2*9.5/M_PI}" soft_lower_limit="${threshold}" soft_upper_limit="${joint_2_limit_soft}" />
 		</joint>
@@ -128,10 +130,11 @@
 		</joint>-->
 		<joint name="${name}_joint_3" type="revolute">
-			<origin xyz="0.000 0.000 0.155" rpy="0 ${146 * M_PI / 180} 0"/>
+<!-- 			<origin xyz="0.000 0.000 0.155" rpy="0 ${146 * M_PI / 180} 0"/> -->
+			<origin xyz="0.000 0.000 0.155" rpy="0 0 0"/>
 			<parent link="${name}_link_2"/>
 			<child link="${name}_link_3"/>
 			<axis xyz="0 1 0"/>
 			<dynamics damping="1" friction="1" />
-			<limit effort="${6}" velocity="${M_PI / 2.0}" lower="-${joint_3_limit}" upper="0"/>
+			<limit effort="${6}" velocity="${M_PI / 2.0}" lower="-${joint_3_limit_low}" upper="${joint_3_limit_high}"/>
                         <safety_controller k_position="20" k_velocity="50" soft_lower_limit="-${joint_3_limit_soft}" soft_upper_limit="-${threshold}" />
 		</joint>
@@ -162,5 +165,5 @@
 		<!-- joint between arm_3_link and arm_4_link -->
 		<joint name="${name}_joint_4" type="revolute">
-			<origin xyz="0.000 0.000 0.135" rpy="0 ${-102.5 * M_PI / 180} 0" />
+			<origin xyz="0.000 0.000 0.135" rpy="0 ${0 * M_PI / 180} 0" />
 			<parent link="${name}_link_3"/>
 			<child link="${name}_link_4"/>
@@ -168,5 +171,5 @@
 			<!--<calibration rising="${arm_4_ref}" falling="${arm_4_ref}"/>-->
 			<dynamics damping="1" friction="1" />
-			<limit effort="${2}" velocity="${M_PI / 2.0}" lower="0" upper="${joint_4_limit}"/>
+			<limit effort="${2}" velocity="${M_PI / 2.0}" lower="${-102.5 * M_PI / 180}" upper="${102.5 * M_PI / 180}"/>
 			<safety_controller k_position="20" k_velocity="100" soft_lower_limit="0" soft_upper_limit="${joint_4_limit_soft}" />
 		</joint>

File: workspaces/youbot/src/youbot_description/urdf/youbot_arm/limits.urdf.xacro (robot description, xacro)
@@ -7,6 +7,12 @@
 	<!-- arm limits positions (deg) -->
 	<property name="joint_1_limit" value="${M_PI * (169 + 169) / 180}" />
+	<property name="joint_1_limit_low" value="${M_PI * (169) / 180}" />
+	<property name="joint_1_limit_high" value="${M_PI * (169) / 180}" />
 	<property name="joint_2_limit" value="${M_PI * (90 + 65) / 180}" />
+	<property name="joint_2_limit_low" value="${M_PI * 65 / 180}" />
+	<property name="joint_2_limit_high" value="${M_PI * 90 / 180}" />
 	<property name="joint_3_limit" value="${M_PI * (146 + 151) / 180}" />
+	<property name="joint_3_limit_low" value="${M_PI * (146) / 180}" />
+	<property name="joint_3_limit_high" value="${M_PI * (151) / 180}" />
 	<property name="joint_4_limit" value="${M_PI * (102.5 + 102.5) / 180}" />
 	<property name="joint_5_limit" value="${M_PI * (167.5 + 167.5) / 180}" />

Commit message: changed arm default joint values such that robot is initilized in 0-position

File: workspaces/youbot/src/youbot_description/urdf/youbot_arm/arm.urdf.xacro (robot description, xacro)
@@ -85,6 +85,6 @@
 		<!-- joint between arm_1_link and arm_2_link -->
 		<joint name="${name}_joint_2" type="revolute">
-<!-- 			<origin xyz="0.033 0 0" rpy="0 ${-65 * M_PI / 180} 0"/> -->
-			<origin xyz="0.033 0 0" rpy="0 ${0 * M_PI / 180} 0"/>
+ 			<origin xyz="0.033 0 0" rpy="0 ${-65 * M_PI / 180} 0"/>
+<!--			<origin xyz="0.033 0 0" rpy="0 ${0 * M_PI / 180} 0"/>-->
 			<parent link="${name}_link_1"/>
 			<child link="${name}_link_2"/>
@@ -92,6 +92,7 @@
 			<!--<calibration rising="${arm_2_ref}" falling="${arm_2_ref}"/>-->
 			<dynamics damping="1" friction="1" />
-			<limit effort="${9.5}" velocity="${M_PI / 2.0}" lower="-${joint_2_limit_low}" upper="${joint_2_limit_high}"/>
-                        <safety_controller k_position="20" k_velocity="${2*9.5/M_PI}" soft_lower_limit="${threshold}" soft_upper_limit="${joint_2_limit_soft}" />
+<!--			<limit effort="${9.5}" velocity="${M_PI / 2.0}" lower="-${joint_2_limit_low}" upper="${joint_2_limit_high}"/>-->
+			<limit effort="${9.5}" velocity="${M_PI / 2.0}" lower="${0}" upper="${joint_2_limit}"/>
+      <safety_controller k_position="20" k_velocity="${2*9.5/M_PI}" soft_lower_limit="${threshold}" soft_upper_limit="${joint_2_limit_soft}" />
 		</joint>
 		<link name="${name}_link_2">
@@ -130,12 +131,13 @@
 		</joint>-->
 		<joint name="${name}_joint_3" type="revolute">
-<!-- 			<origin xyz="0.000 0.000 0.155" rpy="0 ${146 * M_PI / 180} 0"/> -->
-			<origin xyz="0.000 0.000 0.155" rpy="0 0 0"/>
+ 			<origin xyz="0.000 0.000 0.155" rpy="0 ${146 * M_PI / 180} 0"/>
+<!--			<origin xyz="0.000 0.000 0.155" rpy="0 0 0"/>-->
 			<parent link="${name}_link_2"/>
 			<child link="${name}_link_3"/>
 			<axis xyz="0 1 0"/>
 			<dynamics damping="1" friction="1" />
-			<limit effort="${6}" velocity="${M_PI / 2.0}" lower="-${joint_3_limit_low}" upper="${joint_3_limit_high}"/>
-                        <safety_controller k_position="20" k_velocity="50" soft_lower_limit="-${joint_3_limit_soft}" soft_upper_limit="-${threshold}" />
+			<limit effort="${6}" velocity="${M_PI / 2.0}" lower="-${joint_3_limit}" upper="${0}"/>
+<!--			<limit effort="${6}" velocity="${M_PI / 2.0}" lower="-${joint_3_limit_low}" upper="${joint_3_limit_high}"/>-->
+      <safety_controller k_position="20" k_velocity="50" soft_lower_limit="-${joint_3_limit_soft}" soft_upper_limit="-${threshold}" />
 		</joint>
 		<link name="${name}_link_3">
@@ -165,5 +167,6 @@
 		<!-- joint between arm_3_link and arm_4_link -->
 		<joint name="${name}_joint_4" type="revolute">
-			<origin xyz="0.000 0.000 0.135" rpy="0 ${0 * M_PI / 180} 0" />
+<!--			<origin xyz="0.000 0.000 0.135" rpy="0 0 0" />-->
+						<origin xyz="0.000 0.000 0.135" rpy="0 ${102.5 * M_PI / 180} 0" />
 			<parent link="${name}_link_3"/>
 			<child link="${name}_link_4"/>
@@ -171,5 +174,6 @@
 			<!--<calibration rising="${arm_4_ref}" falling="${arm_4_ref}"/>-->
 			<dynamics damping="1" friction="1" />
-			<limit effort="${2}" velocity="${M_PI / 2.0}" lower="${-102.5 * M_PI / 180}" upper="${102.5 * M_PI / 180}"/>
+			<limit effort="${2}" velocity="${M_PI / 2.0}" lower="${0}" upper="${joint_4_limit}"/>
+<!--			<limit effort="${2}" velocity="${M_PI / 2.0}" lower="${-102.5 * M_PI / 180}" upper="${102.5 * M_PI / 180}"/>-->
 			<safety_controller k_position="20" k_velocity="100" soft_lower_limit="0" soft_upper_limit="${joint_4_limit_soft}" />
 		</joint>

Commit message: changed the starting positions of the joints

File: workspaces/youbot/src/youbot_description/urdf/youbot_arm/arm.urdf.xacro (robot description, xacro)
@@ -168,5 +168,5 @@
 		<joint name="${name}_joint_4" type="revolute">
 <!--			<origin xyz="0.000 0.000 0.135" rpy="0 0 0" />-->
-						<origin xyz="0.000 0.000 0.135" rpy="0 ${102.5 * M_PI / 180} 0" />
+						<origin xyz="0.000 0.000 0.135" rpy="0 ${-102.5 * M_PI / 180} 0" />
 			<parent link="${name}_link_3"/>
 			<child link="${name}_link_4"/>
