Commit message: xacro include fix

File: workspaces/youbot/src/youbot_description/urdf/youbot_arm/arm.urdf.xacro (robot description, xacro)
@@ -4,236 +4,236 @@
         xmlns:interface="http://playerstage.sourceforge.net/gazebo/xmlschema/#interface"
         xmlns:xacro="http://ros.org/wiki/xacro">
-	<xacro:include filename="$(find youbot_description)/urdf/youbot_arm/arm.gazebo.xacro" />
-	<xacro:include filename="$(find youbot_description)/urdf/youbot_arm/arm.transmission.xacro" />
+  <xacro:include filename="$(find youbot_description)/urdf/youbot_arm/arm.gazebo.xacro" />
+  <xacro:include filename="$(find youbot_description)/urdf/youbot_arm/arm.transmission.xacro" />
         <xacro:include filename="$(find youbot_description)/urdf/youbot_arm/limits.urdf.xacro" />
-	<xacro:macro name="youbot_arm" params="parent name *origin">
-		<!-- joint between base_link and arm_0_link -->
-		<joint name="${name}_joint_0" type="fixed" >
-			<insert_block name="origin" />
-			<parent link="${parent}" />
-			<child link="${name}_link_0" />
-		</joint>
-		<link name="${name}_link_0">
-			<inertial>
-				<!--<origin xyz="0.023 0 0.006" rpy="0 0 0"/>-->
-				<origin xyz="0 0 0" rpy="0 0 0"/>
-				<mass value="${link_0_mass}"/>
-				<inertia ixx="0.01" ixy="0" ixz="0" iyy="0.01" iyz="0" izz="0.01" />
-			</inertial>
-			<visual>
-				<origin xyz="0 0 0" rpy="0 0 0" />
-				<geometry>
-					<mesh filename="package://youbot_description/meshes/youbot_arm/arm0.dae" />
-				</geometry>
-				<material name="DarkGrey" />
-			</visual>
-			<collision>
-				<!--<origin xyz="0.023 0 0.006" rpy="0 0 0"/>-->
-				<origin xyz="0 0 0" rpy="0 0 0"/>
-				<geometry>
-					<mesh filename="package://youbot_description/meshes/youbot_arm/arm0_convex.dae" />
-					<!--<cylinder length="0.078" radius="0.093"/>-->
-				</geometry>
-			</collision>
-		</link>
-		<gazebo reference = "${name}_link_0">
-			<material>DarkGrey</material>
-		</gazebo>
-		<!-- joint between arm_0_link and arm_1_link -->
-		<joint name="${name}_joint_1" type="revolute">
-			 <origin xyz="0.024 0 0.115" rpy="0 0 ${169 * M_PI / 180}"/>
-<!-- 			<origin xyz="0.024 0 0.115" rpy="0 0 0"/> -->
-			<parent link="${name}_link_0"/>
-			<child link="${name}_link_1"/>
-			<axis xyz="0 0 -1"/>
-			<!--<calibration rising="${arm_1_ref}" falling="${arm_1_ref}"/>-->
-			<dynamics damping="1" friction="1" />
-			<!-- damping - N*s/m, N*s*m/rad -->
-			<!-- friction - N, N*m -->
-			<limit effort="${9.5}" velocity="${M_PI / 2.0}" lower="${0}" upper="${joint_1_limit}"/>
-			<!--effort - N, N*m-->
-			<!--velocity - m/s, rad/s-->
-			<safety_controller k_position="20" k_velocity="${9.5/M_PI / 2.0}" soft_lower_limit="${threshold}" soft_upper_limit="${joint_1_limit_soft}" />
-			<!--k_position N/m, N/rad-->
-			<!--k_velocity N*s/m, N*s*m/rad-->
-			<!--for details: http://www.ros.org/wiki/pr2_controller_manager/safety_limits-->
-		</joint>
-		<link name="${name}_link_1">
-			<inertial>
-				<mass value="${link_1_mass}"/>
-				<xacro:link_1_inertia_tensor />
-			</inertial>
-			<visual>
-				<origin xyz="0 0 0" rpy="${M_PI} 0 0" />
-				<geometry>
-				  <mesh filename="package://youbot_description/meshes/youbot_arm/arm1.dae" />
-				</geometry>
-				<!--<material name="Orange" />-->
-			</visual>
-			<collision>
-				<!--<origin xyz="0 0 -0.003" rpy="0 0 0" />-->
-				<origin xyz="0 0 0" rpy="${M_PI} 0 0" />
-				<geometry>
-					<mesh filename="package://youbot_description/meshes/youbot_arm/arm_joint_1_convex.stl" />
-					<!--<cylinder length="0.102" radius="0.080"/>-->
-				</geometry>
-			</collision>
-		</link>
-		<gazebo reference = "${name}_link_1">
-			<material>Orange</material>
-		</gazebo>
-		<!-- joint between arm_1_link and arm_2_link -->
-		<joint name="${name}_joint_2" type="revolute">
- 			<origin xyz="0.033 0 0" rpy="0 ${-65 * M_PI / 180} 0"/>
-<!--			<origin xyz="0.033 0 0" rpy="0 ${0 * M_PI / 180} 0"/>-->
-			<parent link="${name}_link_1"/>
-			<child link="${name}_link_2"/>
-			<axis xyz="0 1 0"/>
-			<!--<calibration rising="${arm_2_ref}" falling="${arm_2_ref}"/>-->
-			<dynamics damping="1" friction="1" />
-<!--			<limit effort="${9.5}" velocity="${M_PI / 2.0}" lower="-${joint_2_limit_low}" upper="${joint_2_limit_high}"/>-->
-			<limit effort="${9.5}" velocity="${M_PI / 2.0}" lower="${0}" upper="${joint_2_limit}"/>
+  <xacro:macro name="youbot_arm" params="parent name *origin">
+    <!-- joint between base_link and arm_0_link -->
+    <joint name="${name}_joint_0" type="fixed" >
+      <insert_block name="origin" />
+      <parent link="${parent}" />
+      <child link="${name}_link_0" />
+    </joint>
+    <link name="${name}_link_0">
+      <inertial>
+        <!--<origin xyz="0.023 0 0.006" rpy="0 0 0"/>-->
+        <origin xyz="0 0 0" rpy="0 0 0"/>
+        <mass value="${link_0_mass}"/>
+        <inertia ixx="0.01" ixy="0" ixz="0" iyy="0.01" iyz="0" izz="0.01" />
+      </inertial>
+      <visual>
+        <origin xyz="0 0 0" rpy="0 0 0" />
+        <geometry>
+          <mesh filename="package://youbot_description/meshes/youbot_arm/arm0.dae" />
+        </geometry>
+        <material name="DarkGrey" />
+      </visual>
+      <collision>
+        <!--<origin xyz="0.023 0 0.006" rpy="0 0 0"/>-->
+        <origin xyz="0 0 0" rpy="0 0 0"/>
+        <geometry>
+          <mesh filename="package://youbot_description/meshes/youbot_arm/arm0_convex.dae" />
+          <!--<cylinder length="0.078" radius="0.093"/>-->
+        </geometry>
+      </collision>
+    </link>
+    <gazebo reference = "${name}_link_0">
+      <material>DarkGrey</material>
+    </gazebo>
+    <!-- joint between arm_0_link and arm_1_link -->
+    <joint name="${name}_joint_1" type="revolute">
+       <origin xyz="0.024 0 0.115" rpy="0 0 ${169 * M_PI / 180}"/>
+<!--       <origin xyz="0.024 0 0.115" rpy="0 0 0"/> -->
+      <parent link="${name}_link_0"/>
+      <child link="${name}_link_1"/>
+      <axis xyz="0 0 -1"/>
+      <!--<calibration rising="${arm_1_ref}" falling="${arm_1_ref}"/>-->
+      <dynamics damping="1" friction="1" />
+      <!-- damping - N*s/m, N*s*m/rad -->
+      <!-- friction - N, N*m -->
+      <limit effort="${9.5}" velocity="${M_PI / 2.0}" lower="${0}" upper="${joint_1_limit}"/>
+      <!--effort - N, N*m-->
+      <!--velocity - m/s, rad/s-->
+      <safety_controller k_position="20" k_velocity="${9.5/M_PI / 2.0}" soft_lower_limit="${threshold}" soft_upper_limit="${joint_1_limit_soft}" />
+      <!--k_position N/m, N/rad-->
+      <!--k_velocity N*s/m, N*s*m/rad-->
+      <!--for details: http://www.ros.org/wiki/pr2_controller_manager/safety_limits-->
+    </joint>
+    <link name="${name}_link_1">
+      <inertial>
+        <mass value="${link_1_mass}"/>
+        <xacro:link_1_inertia_tensor />
+      </inertial>
+      <visual>
+        <origin xyz="0 0 0" rpy="${M_PI} 0 0" />
+        <geometry>
+          <mesh filename="package://youbot_description/meshes/youbot_arm/arm1.dae" />
+        </geometry>
+        <!--<material name="Orange" />-->
+      </visual>
+      <collision>
+        <!--<origin xyz="0 0 -0.003" rpy="0 0 0" />-->
+        <origin xyz="0 0 0" rpy="${M_PI} 0 0" />
+        <geometry>
+          <mesh filename="package://youbot_description/meshes/youbot_arm/arm_joint_1_convex.stl" />
+          <!--<cylinder length="0.102" radius="0.080"/>-->
+        </geometry>
+      </collision>
+    </link>
+    <gazebo reference = "${name}_link_1">
+      <material>Orange</material>
+    </gazebo>
+    <!-- joint between arm_1_link and arm_2_link -->
+    <joint name="${name}_joint_2" type="revolute">
+       <origin xyz="0.033 0 0" rpy="0 ${-65 * M_PI / 180} 0"/>
+<!--      <origin xyz="0.033 0 0" rpy="0 ${0 * M_PI / 180} 0"/>-->
+      <parent link="${name}_link_1"/>
+      <child link="${name}_link_2"/>
+      <axis xyz="0 1 0"/>
+      <!--<calibration rising="${arm_2_ref}" falling="${arm_2_ref}"/>-->
+      <dynamics damping="1" friction="1" />
+<!--      <limit effort="${9.5}" velocity="${M_PI / 2.0}" lower="-${joint_2_limit_low}" upper="${joint_2_limit_high}"/>-->
+      <limit effort="${9.5}" velocity="${M_PI / 2.0}" lower="${0}" upper="${joint_2_limit}"/>
       <safety_controller k_position="20" k_velocity="${2*9.5/M_PI}" soft_lower_limit="${threshold}" soft_upper_limit="${joint_2_limit_soft}" />
-		</joint>
-		<link name="${name}_link_2">
-			<inertial>
-				<mass value="${link_2_mass}"/>
-				<xacro:link_2_inertia_tensor />
-			</inertial>
-			<visual>
-			<origin xyz="0 0 0" rpy="${- M_PI / 2} ${- M_PI / 2} 0" />
-				<geometry>
-				  <mesh filename="package://youbot_description/meshes/youbot_arm/arm2.dae" />
-				</geometry>
-				<material name="Orange" />
-			</visual>
-			<collision>
-				<!--<origin xyz="0.001 -0.041 0.074" rpy="0 0 0" />-->
-				<origin xyz="0 0 0" rpy="${- M_PI / 2} ${- M_PI / 2} 0" />
-				<geometry>
-					<mesh filename="package://youbot_description/meshes/youbot_arm/arm_joint_2_convex.stl" />
-					<!--<box size="0.074 0.082 0.222"/>-->
-				</geometry>
-			</collision>
-		</link>
-		<gazebo reference = "${name}_link_2">
-			<material>Orange</material>
-		</gazebo>
-		<!-- joint between arm_2_link and arm_3_link -->
-		<!--<joint name="${name}_joint_3" type="revolute">
-			<origin xyz="0.000 0.000 0.155" rpy="0 ${146 * M_PI / 180} 0"/>
-			<parent link="${name}_link_2"/>
-			<child link="${name}_link_3"/>
-			<axis xyz="0 1 0"/>
-			<dynamics damping="1" friction="1" />
-			<limit effort="${6}" velocity="${M_PI / 2.0}" lower="-${joint_3_limit}" upper="0"/>
+    </joint>
+    <link name="${name}_link_2">
+      <inertial>
+        <mass value="${link_2_mass}"/>
+        <xacro:link_2_inertia_tensor />
+      </inertial>
+      <visual>
+      <origin xyz="0 0 0" rpy="${- M_PI / 2} ${- M_PI / 2} 0" />
+        <geometry>
+          <mesh filename="package://youbot_description/meshes/youbot_arm/arm2.dae" />
+        </geometry>
+        <material name="Orange" />
+      </visual>
+      <collision>
+        <!--<origin xyz="0.001 -0.041 0.074" rpy="0 0 0" />-->
+        <origin xyz="0 0 0" rpy="${- M_PI / 2} ${- M_PI / 2} 0" />
+        <geometry>
+          <mesh filename="package://youbot_description/meshes/youbot_arm/arm_joint_2_convex.stl" />
+          <!--<box size="0.074 0.082 0.222"/>-->
+        </geometry>
+      </collision>
+    </link>
+    <gazebo reference = "${name}_link_2">
+      <material>Orange</material>
+    </gazebo>
+    <!-- joint between arm_2_link and arm_3_link -->
+    <!--<joint name="${name}_joint_3" type="revolute">
+      <origin xyz="0.000 0.000 0.155" rpy="0 ${146 * M_PI / 180} 0"/>
+      <parent link="${name}_link_2"/>
+      <child link="${name}_link_3"/>
+      <axis xyz="0 1 0"/>
+      <dynamics damping="1" friction="1" />
+      <limit effort="${6}" velocity="${M_PI / 2.0}" lower="-${joint_3_limit}" upper="0"/>
                         <safety_controller k_position="20" k_velocity="50" soft_lower_limit="-${joint_3_limit_soft}" soft_upper_limit="${threshold}" />
-		</joint>-->
-		<joint name="${name}_joint_3" type="revolute">
- 			<origin xyz="0.000 0.000 0.155" rpy="0 ${146 * M_PI / 180} 0"/>
-<!--			<origin xyz="0.000 0.000 0.155" rpy="0 0 0"/>-->
-			<parent link="${name}_link_2"/>
-			<child link="${name}_link_3"/>
-			<axis xyz="0 1 0"/>
-			<dynamics damping="1" friction="1" />
-			<limit effort="${6}" velocity="${M_PI / 2.0}" lower="-${joint_3_limit}" upper="${0}"/>
-<!--			<limit effort="${6}" velocity="${M_PI / 2.0}" lower="-${joint_3_limit_low}" upper="${joint_3_limit_high}"/>-->
+    </joint>-->
+    <joint name="${name}_joint_3" type="revolute">
+       <origin xyz="0.000 0.000 0.155" rpy="0 ${146 * M_PI / 180} 0"/>
+<!--      <origin xyz="0.000 0.000 0.155" rpy="0 0 0"/>-->
+      <parent link="${name}_link_2"/>
+      <child link="${name}_link_3"/>
+      <axis xyz="0 1 0"/>
+      <dynamics damping="1" friction="1" />
+      <limit effort="${6}" velocity="${M_PI / 2.0}" lower="-${joint_3_limit}" upper="${0}"/>
+<!--      <limit effort="${6}" velocity="${M_PI / 2.0}" lower="-${joint_3_limit_low}" upper="${joint_3_limit_high}"/>-->
       <safety_controller k_position="20" k_velocity="50" soft_lower_limit="-${joint_3_limit_soft}" soft_upper_limit="-${threshold}" />
-		</joint>
-		<link name="${name}_link_3">
-			<inertial>
-				<mass value="${link_3_mass}"/>
-				<xacro:link_3_inertia_tensor />
-			</inertial>
-			<visual>
-				<origin xyz="0 0 0" rpy="${M_PI / 2} 0 ${M_PI}" />
-				<geometry>
-				  <mesh filename="package://youbot_description/meshes/youbot_arm/arm3.dae" />
-				</geometry>
-				<material name="Orange" />
-			</visual>
-			<collision>
-				<!--<origin xyz="0.000 0.025 0.067" rpy="0 0 0" />-->
-				<origin xyz="0 0 0" rpy="${M_PI / 2} 0 ${M_PI}" />
-				<geometry>
-					<mesh filename="package://youbot_description/meshes/youbot_arm/arm_joint_3_convex.stl" />
-					<!--<box size="0.064 0.054 0.192"/>-->
-				</geometry>
-			</collision>
-		</link>
-		<gazebo reference = "${name}_link_3">
-			<material>Orange</material>
-		</gazebo>
-		<!-- joint between arm_3_link and arm_4_link -->
-		<joint name="${name}_joint_4" type="revolute">
-<!--			<origin xyz="0.000 0.000 0.135" rpy="0 0 0" />-->
-						<origin xyz="0.000 0.000 0.135" rpy="0 ${-102.5 * M_PI / 180} 0" />
-			<parent link="${name}_link_3"/>
-			<child link="${name}_link_4"/>
-			<axis xyz="0 1 0" />
-			<!--<calibration rising="${arm_4_ref}" falling="${arm_4_ref}"/>-->
-			<dynamics damping="1" friction="1" />
-			<limit effort="${2}" velocity="${M_PI / 2.0}" lower="${0}" upper="${joint_4_limit}"/>
-<!--			<limit effort="${2}" velocity="${M_PI / 2.0}" lower="${-102.5 * M_PI / 180}" upper="${102.5 * M_PI / 180}"/>-->
-			<safety_controller k_position="20" k_velocity="100" soft_lower_limit="0" soft_upper_limit="${joint_4_limit_soft}" />
-		</joint>
-		<link name="${name}_link_4">
-			<inertial>
-				<mass value="${link_4_mass}"/>
-				<xacro:link_4_inertia_tensor />
-			</inertial>
-			<visual>
-				<origin xyz="0 0 0" rpy="${M_PI / 2} 0 ${M_PI}"/>
-				<geometry>
-				  <mesh filename="package://youbot_description/meshes/youbot_arm/arm4.dae" />
-				</geometry>
-				<material name="Orange" />
-			</visual>
-			<collision>
-				<!--<origin xyz="0 0 0.026" rpy="0 0 0" />-->
-				<origin xyz="0 0 0" rpy="${M_PI / 2} 0 ${M_PI}"/>
-				<geometry>
-					<mesh filename="package://youbot_description/meshes/youbot_arm/arm_joint_4_convex.stl" />
-					<!--<box size="0.058 0.100 0.118"/>-->
-				</geometry>
-			</collision>
-		</link>
-		<gazebo reference = "${name}_link_4">
-			<material>Orange</material>
-		</gazebo>
-		<!-- joint between arm_4_link and arm_5_link -->
-		<joint name="${name}_joint_5" type="revolute">
-			<origin xyz="0 0 0.114" rpy="0 0 ${167.5 * M_PI / 180}" />
-			<parent link="${name}_link_4"/>
-			<child link="${name}_link_5"/>
-			<axis xyz="0 0 -1" />
-			<!--<calibration rising="${arm_5_ref}" falling="${arm_5_ref}"/>-->
-			<dynamics damping="1" friction="1" />
-			<limit effort="1" velocity="${M_PI / 2.0}" lower="0" upper="${joint_5_limit}" />
-                        <safety_controller k_position="20" k_velocity="100" soft_lower_limit="0" soft_upper_limit="${joint_5_limit_soft}" />
-		</joint>
-		<link name="${name}_link_5">
-			<inertial>
-				<mass value="${link_5_mass}"/>
-				<xacro:link_5_inertia_tensor />
-			</inertial>
-			<visual>
-				<origin xyz="0 0 0" rpy="0 0 0" />
-				<geometry>
-				  <mesh filename="package://youbot_description/meshes/youbot_arm/arm5.dae" />
-				</geometry>
-				<material name="DarkGrey" />
-			</visual>
-			<collision>
-				<origin xyz="0 0 0" rpy="0 0 0" />
-				<geometry>
-					<mesh filename="package://youbot_description/meshes/youbot_arm/arm_joint_5_convex.stl" />
-					<!--<box size="0.054 0.096 0.030"/>-->
-				</geometry>
-			</collision>
-		</link>
-		<gazebo reference = "${name}_link_5">
-			<material>DarkGrey</material>
-		</gazebo>
+    </joint>
+    <link name="${name}_link_3">
+      <inertial>
+        <mass value="${link_3_mass}"/>
+        <xacro:link_3_inertia_tensor />
+      </inertial>
+      <visual>
+        <origin xyz="0 0 0" rpy="${M_PI / 2} 0 ${M_PI}" />
+        <geometry>
+          <mesh filename="package://youbot_description/meshes/youbot_arm/arm3.dae" />
+        </geometry>
+        <material name="Orange" />
+      </visual>
+      <collision>
+        <!--<origin xyz="0.000 0.025 0.067" rpy="0 0 0" />-->
+        <origin xyz="0 0 0" rpy="${M_PI / 2} 0 ${M_PI}" />
+        <geometry>
+          <mesh filename="package://youbot_description/meshes/youbot_arm/arm_joint_3_convex.stl" />
+          <!--<box size="0.064 0.054 0.192"/>-->
+        </geometry>
+      </collision>
+    </link>
+    <gazebo reference = "${name}_link_3">
+      <material>Orange</material>
+    </gazebo>
+    <!-- joint between arm_3_link and arm_4_link -->
+    <joint name="${name}_joint_4" type="revolute">
+<!--      <origin xyz="0.000 0.000 0.135" rpy="0 0 0" />-->
+            <origin xyz="0.000 0.000 0.135" rpy="0 ${-102.5 * M_PI / 180} 0" />
+      <parent link="${name}_link_3"/>
+      <child link="${name}_link_4"/>
+      <axis xyz="0 1 0" />
+      <!--<calibration rising="${arm_4_ref}" falling="${arm_4_ref}"/>-->
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